File: gpio-module.kicad_sch (KiCad schematic)
At the start: 0 parts

Commit message: [#1] Init project from base-module template
Other:
- title: ModuCard BM STM32H562VGT6 -> ModuCard GPIO module
Changed lines of the file:
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@@
 	(paper "A4")
 	(title_block
-		(title "ModuCard BM STM32H562VGT6")
-		(date "2025-04-18")
-		(rev "1.1.0")
+		(title "ModuCard GPIO module")
+		(date "2025-04-19")
+		(rev "1.0.0")
 		(company "KoNaR")
 		(comment 1 "Base project authors: Dominik Pluta, Artem Horiunov")
-		(comment 2 "Project author: <author>")
+		(comment 2 "Project author: Dominik Pluta")
 	)
 	(bus_alias "CAN"
@@
 		)
 		(instances
-			(project "base-module"
+			(project "gpio-module"
 				(path "/090a8e41-87a8-4fb1-998b-60a2c0dc4cee"
 					(page "6")
@@
 		)
 		(instances
-			(project "base-module"
+			(project "gpio-module"
 				(path "/090a8e41-87a8-4fb1-998b-60a2c0dc4cee"
 					(page "3")
@@
 		)
 		(instances
-			(project "base-module"
+			(project "gpio-module"
 				(path "/090a8e41-87a8-4fb1-998b-60a2c0dc4cee"
 					(page "5")
@@
 		)
 		(instances
-			(project "base-module"
+			(project "gpio-module"
 				(path "/090a8e41-87a8-4fb1-998b-60a2c0dc4cee"
 					(page "8")
@@
 		)
 		(instances
-			(project "base-module"
+			(project "gpio-module"
 				(path "/090a8e41-87a8-4fb1-998b-60a2c0dc4cee"
 					(page "4")
@@
 		)
 		(instances
-			(project "base-module"
+			(project "gpio-module"
 				(path "/090a8e41-87a8-4fb1-998b-60a2c0dc4cee"
 					(page "9")
@@
 		)
 		(instances
-			(project "base-module"
+			(project "gpio-module"
 				(path "/090a8e41-87a8-4fb1-998b-60a2c0dc4cee"
 					(page "10")
@@
 		)
 		(instances
-			(project "base-module"
+			(project "gpio-module"
 				(path "/090a8e41-87a8-4fb1-998b-60a2c0dc4cee"
 					(page "7")
@@
 		)
 		(instances
-			(project "base-module"
+			(project "gpio-module"
 				(path "/090a8e41-87a8-4fb1-998b-60a2c0dc4cee"
 					(page "2")

Commit message: [#1] Add LED connector and GPIO connectors, place connectors on PCB
Other:
- added sheet GPIO connector (gpio-connector.kicad_sch)
- added sheet GPIO connector1 (gpio-connector.kicad_sch)
- added sheet GPIO connector2 (gpio-connector.kicad_sch)
- added sheet RGB LED connector (rgb-led-connector.kicad_sch)

Commit message: [#1] Connect LED connector to MCU
Other:
- sheet MCU ports: added EXT_LED_B, EXT_LED_G, EXT_LED_R; removed none
Changed lines of the file:
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@@
+		)
+	)
+	(wire
+		(pts
+			(xy 205.74 44.45) (xy 223.52 44.45)
+		)
+		(stroke
+			(width 0)
+			(type default)
 		)
 	)
@@
 		)
 	)
+	(wire
+		(pts
+			(xy 205.74 46.99) (xy 223.52 46.99)
+		)
+		(stroke
+			(width 0)
+			(type default)
+		)
+	)
 	(bus
 		(pts
@@
 		(pts
 			(xy 106.68 49.53) (xy 123.19 49.53)
+		)
+		(stroke
+			(width 0)
+			(type default)
+		)
+	)
+	(wire
+		(pts
+			(xy 205.74 49.53) (xy 223.52 49.53)
 		)
 		(stroke
@@
 			)
 		)
+		(pin "EXT_LED_B" output
+			(at 205.74 49.53 0)
+			(effects
+				(font
+					(size 1.27 1.27)
+				)
+				(justify right)
+			)
+		)
+		(pin "EXT_LED_G" output
+			(at 205.74 46.99 0)
+			(effects
+				(font
+					(size 1.27 1.27)
+				)
+				(justify right)
+			)
+		)
+		(pin "EXT_LED_R" output
+			(at 205.74 44.45 0)
+			(effects
+				(font
+					(size 1.27 1.27)
+				)
+				(justify right)
+			)
+		)

Commit message: [#1] Connect all GPIO connectors to MCU
Other:
- sheet GPIO connector renamed GPIO connector 0
- sheet GPIO connector1 renamed GPIO connector 1
- sheet GPIO connector2 renamed GPIO connector 2
- sheet MCU ports: added GPIO_0_IN, GPIO_0_OUT, GPIO_1_IN, GPIO_1_OUT, GPIO_2_IN, GPIO_2_OUT; removed none
Changed lines of the file:
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@@
+		)
+	)
+	(wire
+		(pts
+			(xy 205.74 74.93) (xy 223.52 74.93)
+		)
+		(stroke
+			(width 0)
+			(type default)
+		)
+	)
+	(wire
+		(pts
+			(xy 205.74 91.44) (xy 223.52 91.44)
+		)
+		(stroke
+			(width 0)
+			(type default)
 		)
 	)
@@
 		)
 	)
+	(wire
+		(pts
+			(xy 205.74 77.47) (xy 223.52 77.47)
+		)
+		(stroke
+			(width 0)
+			(type default)
+		)
+	)
 	(bus
 		(pts
@@
 		)
 	)
+	(wire
+		(pts
+			(xy 205.74 60.96) (xy 223.52 60.96)
+		)
+		(stroke
+			(width 0)
+			(type default)
+		)
+	)
 	(bus
 		(pts
@@
 		)
 	)
+	(wire
+		(pts
+			(xy 205.74 63.5) (xy 223.52 63.5)
+		)
+		(stroke
+			(width 0)
+			(type default)
+		)
+	)
 	(bus
 		(pts
@@
 		(pts
 			(xy 148.59 88.9) (xy 161.29 88.9)
+		)
+		(stroke
+			(width 0)
+			(type default)
+		)
+	)
+	(wire
+		(pts
+			(xy 205.74 88.9) (xy 223.52 88.9)
 		)
 		(stroke
@@
 			(color 0 0 0 0.0000)
 		)
-		(property "Sheetname" "GPIO connector"
+		(property "Sheetname" "GPIO connector 0"
 			(at 223.52 57.7084 0)
 			(effects
@@
 			(color 0 0 0 0.0000)
 		)
-		(property "Sheetname" "GPIO connector1"
+		(property "Sheetname" "GPIO connector 1"
 			(at 223.52 71.6784 0)
 			(effects
@@
 			)
 		)
+		(pin "GPIO_0_IN" input
+			(at 205.74 60.96 0)
+			(effects
+				(font
+					(size 1.27 1.27)
+				)
+				(justify right)
+			)
+		)
+		(pin "GPIO_0_OUT" output
+			(at 205.74 63.5 0)
+			(effects
+				(font
+					(size 1.27 1.27)
+				)
+				(justify right)
+			)
+		)
+		(pin "GPIO_1_IN" input
+			(at 205.74 74.93 0)
+			(effects
+				(font
+					(size 1.27 1.27)
+				)
+				(justify right)
+			)
+		)
+		(pin "GPIO_1_OUT" input
+			(at 205.74 77.47 0)
+			(effects
+				(font
+					(size 1.27 1.27)
+				)
+				(justify right)
+			)
+		)
+		(pin "GPIO_2_IN" input
+			(at 205.74 88.9 0)
+			(effects
+				(font
+					(size 1.27 1.27)
+				)
+				(justify right)
+			)
+		)
+		(pin "GPIO_2_OUT" input
+			(at 205.74 91.44 0)
+			(effects
+				(font
+					(size 1.27 1.27)
+				)
+				(justify right)
+			)
+		)
 		(instances
 			(project "gpio-module"
@@
 			(color 0 0 0 0.0000)
 		)
-		(property "Sheetname" "GPIO connector2"
+		(property "Sheetname" "GPIO connector 2"
 			(at 223.52 85.6484 0)
 			(effects

Commit message: [#1] Connect GPIOR to MCU
Connections:
- no-connect marks 3 -> 1
Other:
- sheet MCU ports: added GPIOR[0..15]; removed none
Changed lines of the file:
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@@
 		(at 81.28 82.55)
 	)
-	(no_connect
-		(at 81.28 88.9)
-	)
-	(no_connect
-		(at 81.28 96.52)
-	)
 	(bus
 		(pts
@@
 		)
 	)
+	(bus
+		(pts
+			(xy 184.15 140.97) (xy 184.15 165.1)
+		)
+		(stroke
+			(width 0)
+			(type default)
+		)
+	)
 	(wire
 		(pts
@@
 		)
 	)
+	(bus
+		(pts
+			(xy 74.93 165.1) (xy 74.93 96.52)
+		)
+		(stroke
+			(width 0)
+			(type default)
+		)
+	)
 	(wire
 		(pts
@@
 	(bus
 		(pts
+			(xy 74.93 96.52) (xy 81.28 96.52)
+		)
+		(stroke
+			(width 0)
+			(type default)
+		)
+	)
+	(bus
+		(pts
 			(xy 148.59 137.16) (xy 161.29 137.16)
 		)
@@
 		(pts
 			(xy 205.74 60.96) (xy 223.52 60.96)
+		)
+		(stroke
+			(width 0)
+			(type default)
+		)
+	)
+	(bus
+		(pts
+			(xy 184.15 165.1) (xy 74.93 165.1)
 		)
 		(stroke
@@
 			)
 		)
+		(pin "GPIOR[0..15]" input
+			(at 184.15 140.97 270)
+			(effects
+				(font
+					(size 1.27 1.27)
+				)
+				(justify left)
+			)
+		)

Commit message: [#1] Connect 12V to front connectors, connect GPIOL to MCU
Other:
- sheet MCU ports: added GPIOL[0..15]; removed none
Changed lines of the file:
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@@
+		)
+	)
+	(bus
+		(pts
+			(xy 208.28 161.29) (xy 208.28 137.16)
+		)
+		(stroke
+			(width 0)
+			(type default)
 		)
 	)
@@
 		)
 	)
+	(bus
+		(pts
+			(xy 210.82 134.62) (xy 210.82 163.83)
+		)
+		(stroke
+			(width 0)
+			(type default)
+		)
+	)
 	(wire
 		(pts
@@
 		)
 	)
-	(bus
-		(pts
-			(xy 184.15 140.97) (xy 184.15 165.1)
-		)
-		(stroke
-			(width 0)
-			(type default)
-		)
-	)
 	(wire
 		(pts
@@
 	(bus
 		(pts
-			(xy 74.93 165.1) (xy 74.93 96.52)
+			(xy 71.12 88.9) (xy 71.12 163.83)
+		)
+		(stroke
+			(width 0)
+			(type default)
+		)
+	)
+	(bus
+		(pts
+			(xy 81.28 88.9) (xy 71.12 88.9)
+		)
+		(stroke
+			(width 0)
+			(type default)
+		)
+	)
+	(bus
+		(pts
+			(xy 73.66 161.29) (xy 73.66 96.52)
 		)
 		(stroke
@@
 	(bus
 		(pts
-			(xy 74.93 96.52) (xy 81.28 96.52)
+			(xy 73.66 96.52) (xy 81.28 96.52)
 		)
 		(stroke
@@
 		)
 	)
+	(bus
+		(pts
+			(xy 208.28 137.16) (xy 205.74 137.16)
+		)
+		(stroke
+			(width 0)
+			(type default)
+		)
+	)
+	(bus
+		(pts
+			(xy 71.12 163.83) (xy 210.82 163.83)
+		)
+		(stroke
+			(width 0)
+			(type default)
+		)
+	)
 	(wire
 		(pts
@@
 	(bus
 		(pts
-			(xy 184.15 165.1) (xy 74.93 165.1)
+			(xy 208.28 161.29) (xy 73.66 161.29)
+		)
+		(stroke
+			(width 0)
+			(type default)
+		)
+	)
+	(bus
+		(pts
+			(xy 205.74 134.62) (xy 210.82 134.62)
 		)
 		(stroke
@@
 		)
 		(pin "GPIOR[0..15]" input
-			(at 184.15 140.97 270)
-			(effects
-				(font
-					(size 1.27 1.27)
-				)
-				(justify left)
-			)
-		)
+			(at 205.74 137.16 0)
+			(effects
+				(font
+					(size 1.27 1.27)
+				)
+				(justify right)
+			)
+		)
+		(pin "GPIOL[0..15]" input
+			(at 205.74 134.62 0)
+			(effects
+				(font
+					(size 1.27 1.27)
+				)
+				(justify right)
+			)
+		)

Commit message: Replace RGB with CH3 and adjust silk
Other:
- removed sheet RGB LED connector
- added sheet GPIO connector 3 (gpio-connector.kicad_sch)
- sheet MCU ports: added GPIO_3_IN, GPIO_3_OUT; removed EXT_LED_B, EXT_LED_G, EXT_LED_R
