File: gpio-module.kicad_sch (KiCad schematic)
At the start: 0 parts

Commit message: [#6] Define ADC pins, start rerouting
Changed lines of the file:
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@@
 			)
 		)
-		(pin "GPIO_1_OUT" input
+		(pin "GPIO_1_OUT" output
 			(at 205.74 60.96 0)
 			(effects
@@
 			)
 		)
-		(pin "GPIO_2_OUT" input
+		(pin "GPIO_2_OUT" output
 			(at 205.74 74.93 0)
 			(effects
@@
 			)
 		)
-		(pin "GPIO_3_IN" output
+		(pin "GPIO_3_IN" input
 			(at 205.74 86.36 0)
 			(effects

Commit message: [#6] WIP: connect GPIO
Changed lines of the file:
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@@
 	(bus
 		(pts
-			(xy 218.44 137.16) (xy 218.44 165.1)
+			(xy 218.44 137.16) (xy 218.44 161.29)
 		)
 		(stroke
@@
 	(bus
 		(pts
-			(xy 218.44 165.1) (xy 72.39 165.1)
+			(xy 218.44 161.29) (xy 72.39 161.29)
 		)
 		(stroke
@@
 	(bus
 		(pts
-			(xy 72.39 165.1) (xy 72.39 96.52)
+			(xy 72.39 161.29) (xy 72.39 96.52)
 		)
 		(stroke
@@
 		)
 		(instances
-			(project "base-module"
+			(project "gpio-module"
 				(path "/090a8e41-87a8-4fb1-998b-60a2c0dc4cee"
 					(page "6")
@@
 		)
 		(instances
-			(project "base-module"
+			(project "gpio-module"
 				(path "/090a8e41-87a8-4fb1-998b-60a2c0dc4cee"
 					(page "13")
@@
 		)
 		(instances
-			(project "base-module"
+			(project "gpio-module"
 				(path "/090a8e41-87a8-4fb1-998b-60a2c0dc4cee"
 					(page "17")
@@
 		)
 		(instances
-			(project "base-module"
+			(project "gpio-module"
 				(path "/090a8e41-87a8-4fb1-998b-60a2c0dc4cee"
 					(page "3")
@@
 		)
 		(instances
-			(project "base-module"
+			(project "gpio-module"
 				(path "/090a8e41-87a8-4fb1-998b-60a2c0dc4cee"
 					(page "5")
@@
 		)
 		(instances
-			(project "base-module"
+			(project "gpio-module"
 				(path "/090a8e41-87a8-4fb1-998b-60a2c0dc4cee"
 					(page "11")
@@
 		)
 		(instances
-			(project "base-module"
+			(project "gpio-module"
 				(path "/090a8e41-87a8-4fb1-998b-60a2c0dc4cee"
 					(page "15")
@@
 		)
 		(instances
-			(project "base-module"
+			(project "gpio-module"
 				(path "/090a8e41-87a8-4fb1-998b-60a2c0dc4cee"
 					(page "8")
@@
 		)
 		(instances
-			(project "base-module"
+			(project "gpio-module"
 				(path "/090a8e41-87a8-4fb1-998b-60a2c0dc4cee"
 					(page "4")
@@
 		)
 		(instances
-			(project "base-module"
+			(project "gpio-module"
 				(path "/090a8e41-87a8-4fb1-998b-60a2c0dc4cee"
 					(page "9")
@@
 		)
 		(instances
-			(project "base-module"
+			(project "gpio-module"
 				(path "/090a8e41-87a8-4fb1-998b-60a2c0dc4cee"
 					(page "10")
@@
 		)
 		(instances
-			(project "base-module"
+			(project "gpio-module"
 				(path "/090a8e41-87a8-4fb1-998b-60a2c0dc4cee"
 					(page "7")
@@
 		)
 		(instances
-			(project "base-module"
+			(project "gpio-module"
 				(path "/090a8e41-87a8-4fb1-998b-60a2c0dc4cee"
 					(page "2")
