File: power.kicad_sch (KiCad schematic)
At the start: 33 parts, among them U300 TPS563200, U301 TPS563200

Commit message: [#1] Init project using the template - base module project
Other:
- title: ModuCard BM STM32H562VGT6 -> ModuCard GPIO module
Changed lines of the file:
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@@
 	(paper "A4")
 	(title_block
-		(title "ModuCard BM STM32H562VGT6")
-		(date "2025-04-18")
+		(title "ModuCard GPIO module")
+		(date "2025-04-19")
 		(rev "1.0.0")
 		(company "KoNaR")
 		(comment 1 "Base project authors: Dominik Pluta, Artem Horiunov")
-		(comment 2 "Project author: <author>")
+		(comment 2 "Project author: Dominik Pluta")
 	)
 	(rectangle
