File: power.kicad_sch (KiCad schematic)
At the start: 33 parts, among them U300 TPS563200, U301 TPS563200

Commit message: [#8] Fix missing component values, fix soldermask expansion of U800 and remove its designator from silkscreen, minor schematic fixes
Parts:
- removed F300: Fuse, PCM_JLCPCB:R_0603, symbol Device:Fuse
- added F300: 1.5A, PCM_JLCPCB:F_0603, symbol PCM_JLCPCB-Variable-Resistors:Fuse,1.5A
- L300, L301: value L -> 3.3uH
- R300: value R_Small -> 54k9
- R306: value R_Small -> 33k2
Connections:
- net +12V: now also F300.1
- net +12V_FUSED: now also F300.2

Commit message: [#1] Fill out schematic title block, connect GPIOs on the schematic
Other:
- title: ModuCard BM STM32H562VGT6 -> ModuCard GPIO module
Changed lines of the file:
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@@
 	(paper "A4")
 	(title_block
-		(title "ModuCard BM STM32H562VGT6")
-		(date "2025-04-18")
-		(rev "1.1.1")
+		(title "ModuCard GPIO module")
+		(date "2025-06-19")
+		(rev "1.0.0")
 		(company "KoNaR")
 		(comment 1 "Base project authors: Dominik Pluta, Artem Horiunov")
-		(comment 2 "Project author: <author>")
+		(comment 2 "Project author: Dominik Pluta")
 	)
 	(rectangle

Commit message: [#1] Finish PCB
Parts:
- added F301: Fuse, PCM_JLCPCB:R_0603, symbol Device:Fuse
- added TP303: TestPoint, TestPoint:TestPoint_Pad_D1.0mm, symbol Connector:TestPoint
Connections:
- net +12V: now also F301.1
- new net +12V_GPIO: F301.2, TP303.1
