File: st-link.kicad_sch (KiCad schematic)
At the start: 38 parts, among them Q700 MMST3904, U700 STM32F103CBTx, Y700 Crystal_GND24

Commit message: [#1] Init project using the template - base module project
Other:
- title: ModuCard BM STM32H562VGT6 -> ModuCard GPIO module
Changed lines of the file:
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@@
 	(paper "A4")
 	(title_block
-		(title "ModuCard BM STM32H562VGT6")
-		(date "2025-04-18")
+		(title "ModuCard GPIO module")
+		(date "2025-04-19")
 		(rev "1.0.0")
 		(company "KoNaR")
 		(comment 1 "Base project authors: Dominik Pluta, Artem Horiunov")
-		(comment 2 "Project author: <author>")
+		(comment 2 "Project author: Dominik Pluta")
 	)
 	(rectangle
