File: st-link.kicad_sch (KiCad schematic)
At the start: 38 parts, among them Q700 MMST3904, U700 STM32F103CBTx, Y700 Crystal_GND24

Commit message: [#8] Fix missing component values, fix soldermask expansion of U800 and remove its designator from silkscreen, minor schematic fixes
Parts:
- removed R712: 1.2kΩ, PCM_JLCPCB:R_0402, symbol PCM_JLCPCB-Resistors:0402,1.2kΩ
- added R712: 1.5kΩ, PCM_JLCPCB:R_0402, symbol PCM_JLCPCB-Resistors:0402,1.5kΩ
- Y700: value Crystal_GND24 -> 8 MHz
Connections:
- net ST-LINK.D+: now also R712.2
- net at Q700.2 (E): now also R712.1
Other:
- note removed: "Do weryfikackji"
- note removed: "Should be 1k5, but we try 1k2 because it is in basic parts"
Changed lines of the file:
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@@
 		)
 	)
-	(text "Do weryfikackji"
-		(exclude_from_sim no)
-		(at 121.92 151.892 0)
-		(effects
-			(font
-				(size 6 6)
-				(thickness 0.254)
-				(bold yes)
-				(color 255 0 27 1)
-			)
-		)
-	)
-	(text "Should be 1k5,\nbut we try 1k2\nbecause it is in\nbasic parts"
-		(exclude_from_sim no)
-		(at 250.825 122.555 0)
-		(effects
-			(font
-				(size 1.27 1.27)
-				(color 255 0 11 1)
-			)
-		)
-	)
 	(text "ACTIVITY LED\n"
 		(exclude_from_sim no)
@@
 		)
 	)
-	(polyline
-		(pts
-			(xy 242.57 119.38) (xy 232.41 114.3)
-		)
-		(stroke
-			(width 0)
-			(type default)
-		)
-	)
 	(wire
 		(pts
@@
 	(wire
 		(pts
-			(xy 39.37 77.47) (xy 43.18 77.47)
-		)
-		(stroke
-			(width 0)
-			(type default)
-		)
-	)
-	(wire
-		(pts
 			(xy 74.93 57.15) (xy 83.82 57.15)
 		)
@@
 	(polyline
 		(pts
-			(xy 109.22 58.42) (xy 109.22 60.96)
+			(xy 109.22 55.88) (xy 109.22 58.42)
 		)
 		(stroke
@@
 		)
 	)
-	(polyline
-		(pts
-			(xy 232.41 114.3) (xy 233.68 116.84)
-		)
-		(stroke
-			(width 0)
-			(type default)
-		)
-	)
 	(wire
 		(pts
@@
 	(wire
 		(pts
-			(xy 43.18 77.47) (xy 43.18 78.74)
-		)
-		(stroke
-			(width 0)
-			(type default)
-		)
-	)
-	(wire
-		(pts
 			(xy 74.93 46.99) (xy 83.82 46.99)
 		)
@@
 		)
 	)
-	(polyline
-		(pts
-			(xy 232.41 114.3) (xy 234.95 114.3)
-		)
-		(stroke
-			(width 0)
-			(type default)
-		)
-	)
 	(wire
 		(pts
@@
 	(polyline
 		(pts
-			(xy 109.22 60.96) (xy 111.76 59.69)
+			(xy 109.22 58.42) (xy 111.76 57.15)
 		)
 		(stroke
@@
 	(wire
 		(pts
-			(xy 39.37 85.09) (xy 39.37 77.47)
-		)
-		(stroke
-			(width 0)
-			(type default)
-		)
-	)
-	(wire
-		(pts
 			(xy 39.37 46.99) (xy 48.26 46.99)
 		)
@@
 	(wire
 		(pts
-			(xy 123.19 78.74) (xy 124.46 78.74)
+			(xy 123.19 78.74) (xy 134.62 78.74)
 		)
 		(stroke
@@
 	(polyline
 		(pts
-			(xy 118.11 52.07) (xy 109.22 60.96)
+			(xy 118.11 49.53) (xy 109.22 58.42)
 		)
 		(stroke
@@
 	)
 	(label "SWD.SWCLK"
-		(at 124.46 78.74 0)
+		(at 134.62 78.74 180)
 		(effects
 			(font
 				(size 1.27 1.27)
 			)
-			(justify left bottom)
+			(justify right bottom)
 		)
 	)
@@
 	)
 	(symbol
-		(lib_id "PCM_JLCPCB-Resistors:0402,1.2kΩ")
+		(lib_id "PCM_JLCPCB-Resistors:0402,1.5kΩ")
 		(at 229.87 111.76 0)
 		(unit 1)
@@
 			)
 		)
-		(property "Value" "1.2kΩ"
+		(property "Value" "1.5kΩ"
 			(at 229.87 111.76 90)
 			(do_not_autoplace yes)
@@
 			)
 		)
-		(property "Datasheet" "https://www.lcsc.com/datasheet/lcsc_datasheet_2206010045_UNI-ROYAL-Uniroyal-Elec-0402WGF1201TCE_C25862.pdf"
+		(property "Datasheet" "https://www.lcsc.com/datasheet/lcsc_datasheet_2206010045_UNI-ROYAL-Uniroyal-Elec-0402WGF1501TCE_C25867.pdf"
 			(at 229.87 111.76 0)
 			(effects
@@
 			)
 		)
-		(property "Description" "62.5mW Thick Film Resistors 50V ±100ppm/°C ±1% 1.2kΩ 0402 Chip Resistor - Surface Mount ROHS"
+		(property "Description" "62.5mW Thick Film Resistors 50V ±100ppm/°C ±1% 1.5kΩ 0402 Chip Resistor - Surface Mount ROHS"
 			(at 229.87 111.76 0)
 			(effects
@@
 			)
 		)
-		(property "LCSC" "C25862"
+		(property "LCSC" "C25867"
 			(at 229.87 111.76 0)
 			(effects
@@
 			)
 		)
-		(property "Stock" "191144"
+		(property "Stock" "853285"
 			(at 229.87 111.76 0)
 			(effects
@@
 			)
 		)
-		(property "Class" "Preferred Component"
+		(property "Class" "Basic Component"
 			(at 229.87 111.76 0)
 			(effects
@@
 			)
 		)
-		(property "Part" "0402WGF1201TCE"
+		(property "Part" "0402WGF1501TCE"
 			(at 229.87 111.76 0)
 			(effects
@@
 			)
 		)
-		(property "Resistance" "1.2kΩ"
+		(property "Resistance" "1.5kΩ"
 			(at 229.87 111.76 0)
 			(effects
@@
 			)
 		)
-		(pin "1"
-		)
 		(pin "2"
 		)
+		(pin "1"
+		)
 		(instances
-			(project "base-module"
+			(project ""
 				(path "/090a8e41-87a8-4fb1-998b-60a2c0dc4cee/ed5910e5-42de-4923-b023-9e23a66937d0"
 					(reference "R712")
@@
 		(fields_autoplaced yes)
 		(property "Reference" "TP704"
-			(at 207.01 100.9649 90)
+			(at 207.01 101.5999 90)
 			(effects
 				(font
@@
 				)
 				(justify left)
+				(hide yes)
 			)
 		)
@@
 	)
 	(symbol
-		(lib_id "power:GND")
-		(at 43.18 78.74 0)
-		(unit 1)
-		(exclude_from_sim no)
-		(in_bom yes)
-		(on_board yes)
-		(dnp no)
-		(fields_autoplaced yes)
-		(property "Reference" "#PWR0400"
-			(at 43.18 85.09 0)
-			(effects
-				(font
-					(size 1.27 1.27)
-				)
-				(hide yes)
-			)
-		)
-		(property "Value" "GND"
-			(at 43.18 83.82 0)
-			(effects
-				(font
-					(size 1.27 1.27)
-				)
-			)
-		)
-		(property "Footprint" ""
-			(at 43.18 78.74 0)
-			(effects
-				(font
-					(size 1.27 1.27)
-				)
-				(hide yes)
-			)
-		)
-		(property "Datasheet" ""
-			(at 43.18 78.74 0)
-			(effects
-				(font
-					(size 1.27 1.27)
-				)
-				(hide yes)
-			)
-		)
-		(property "Description" "Power symbol creates a global label with name \"GND\" , ground"
-			(at 43.18 78.74 0)
-			(effects
-				(font
-					(size 1.27 1.27)
-				)
-				(hide yes)
-			)
-		)
-		(pin "1"
-		)
-		(instances
-			(project ""
-				(path "/090a8e41-87a8-4fb1-998b-60a2c0dc4cee/ed5910e5-42de-4923-b023-9e23a66937d0"
-					(reference "#PWR0400")
-					(unit 1)
-				)
-			)
-		)
-	)
-	(symbol
 		(lib_id "PCM_JLCPCB-Capacitors:0402,100nF,(2)")
 		(at 74.93 52.07 0)
@@
 		(fields_autoplaced yes)
 		(property "Reference" "TP705"
-			(at 207.01 104.7749 90)
+			(at 207.01 105.4099 90)
 			(effects
 				(font
@@
 				)
 				(justify left)
+				(hide yes)
 			)
 		)
@@
 		(fields_autoplaced yes)
 		(property "Reference" "U700"
-			(at 101.2541 137.16 0)
+			(at 101.2033 139.7 0)
 			(effects
 				(font
@@
 		)
 		(property "Value" "STM32F103CBTx"
-			(at 101.2541 139.7 0)
+			(at 101.2033 142.24 0)
 			(effects
 				(font
@@
 		(fields_autoplaced yes)
 		(property "Reference" "TP702"
-			(at 207.01 93.3449 90)
+			(at 207.01 93.9799 90)
 			(effects
 				(font
@@
 				)
 				(justify left)
+				(hide yes)
 			)
 		)
@@
 		(fields_autoplaced yes)
 		(property "Reference" "TP703"
-			(at 207.01 97.1549 90)
+			(at 207.01 97.7899 90)
 			(effects
 				(font
@@
 				)
 				(justify left)
+				(hide yes)
 			)
 		)
@@
 		(fields_autoplaced yes)
 		(property "Reference" "TP706"
-			(at 207.01 108.5849 90)
+			(at 207.01 109.2199 90)
 			(effects
 				(font
@@
 				)
 				(justify left)
+				(hide yes)
 			)
 		)
@@
 		(dnp no)
 		(property "Reference" "Y700"
-			(at 24.384 87.122 0)
+			(at 39.37 83.312 0)
 			(effects
 				(font
@@
 			)
 		)
-		(property "Value" "Crystal_GND24"
-			(at 24.384 88.9 0)
+		(property "Value" "8 MHz"
+			(at 39.37 85.09 0)
 			(effects
 				(font
@@
 			)
 		)
-		(property "Description" "Four pin crystal, GND on pins 2 and 4"
+		(property "Description" "8MHz 20pF ±10ppm SMD3225 Crystals ROHS"
 			(at 39.37 90.17 0)
 			(effects
@@
 		)
 		(instances
-			(project ""
-				(path "/090a8e41-87a8-4fb1-998b-60a2c0dc4cee/ae074854-c02c-496b-964f-ecb8956e53f8"
-					(reference "Y700")
-					(unit 1)
-				)
+			(project "base-module"
 				(path "/090a8e41-87a8-4fb1-998b-60a2c0dc4cee/ed5910e5-42de-4923-b023-9e23a66937d0"
 					(reference "Y700")

Commit message: [#1] Fill out schematic title block, connect GPIOs on the schematic
Other:
- title: ModuCard BM STM32H562VGT6 -> ModuCard GPIO module
Changed lines of the file:
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@@
 	(paper "A4")
 	(title_block
-		(title "ModuCard BM STM32H562VGT6")
-		(date "2025-04-18")
-		(rev "1.1.1")
+		(title "ModuCard GPIO module")
+		(date "2025-06-19")
+		(rev "1.0.0")
 		(company "KoNaR")
 		(comment 1 "Base project authors: Dominik Pluta, Artem Horiunov")
-		(comment 2 "Project author: <author>")
+		(comment 2 "Project author: Dominik Pluta")
 	)
 	(rectangle
