File: gpio-module.kicad_pcb (KiCad board)
At the start: 4 copper layers, 100 x 100 mm, 166 parts, among them J200 09031967921, J800 USB_C_Receptacle_USB2.0_16P, Q700 MMST3904, U100 W25Q128, U300 TPS563200, U301 TPS563200, U302 CH334P, U401 TPD2E2U06DCK, U402 TPD2E2U06DCK, U403 STM32H562VGTx, U500 TJA1044GTK_3Z, U600 TJA1044GTK_3Z, U700 STM32F103CBTx, U801 FSUSB42UMX, X300 Q13FC1350000400, Y400 ASE-xxxMHz, Y700 Crystal_GND24, Y900 Crystal_GND24

Commit message: [#1] Init project from base-module template
Other:
- board text removed: "* HIGH PERFORMANCE MCU * ADDITIONAL (Q)SPI FLASH * BUILT IN USB DEBUGGER * HIGH SPEED CAN TANSCEIVERS * HIGH POWER 24W VRM"
- board text removed: "1. Add $Project Author$ field 2. Add board revision 3. Remove this silkscreen 4. Layout board 6. Pass DRC 5. Add boardhouse info in designted spot on bottom side"
- board text removed: "BY NOMAD ELECTRONICS TEAM"
- board text removed: "FEATURES:"
- board text removed: "Template Project"
- board text removed: "USAGE:"
- board text removed: "USER AREA"
- board text removed: "predefined area"

Commit message: [#1] Add LED connector and GPIO connectors, place connectors on PCB
Parts:
- added J10: Molex_Micro-Fit_3.0 2x2, Connector_Molex:Molex_Micro-Fit_3.0_43045-0400_2x02_P3.00mm_Horizontal, F.Cu at (66.1, 60.5)
- added J11: Molex_Micro-Fit_3.0 2x2, Connector_Molex:Molex_Micro-Fit_3.0_43045-0400_2x02_P3.00mm_Horizontal, F.Cu at (54.9, 60.5)
- added J8: Molex_Micro-Fit_3.0 2x2, Connector_Molex:Molex_Micro-Fit_3.0_43045-0400_2x02_P3.00mm_Horizontal, F.Cu at (88.7, 60.5)
- added J9: Molex_Micro-Fit_3.0 2x2, Connector_Molex:Molex_Micro-Fit_3.0_43045-0400_2x02_P3.00mm_Horizontal, F.Cu at (77.4, 60.5)
- added Q401: AO3400A, PCM_JLCPCB:Q_SOT-23, F.Cu at (86.8, 69.5)
- added Q402: AO3400A, PCM_JLCPCB:Q_SOT-23, F.Cu at (90.2, 69.5)
- added Q403: AO3400A, PCM_JLCPCB:Q_SOT-23, F.Cu at (93.6, 69.5)
- added Q405: AO3400A, PCM_JLCPCB:Q_SOT-23, F.Cu at (80.4, 69.5)
- added Q406: AO3400A, PCM_JLCPCB:Q_SOT-23, F.Cu at (69.1, 69.5)
- added Q407: AO3400A, PCM_JLCPCB:Q_SOT-23, F.Cu at (57.9, 69.5)
- added R413: 10kΩ, PCM_JLCPCB:R_0402, F.Cu at (86.8, 71.9)
- added R414: 0Ω, PCM_JLCPCB:R_0402, F.Cu at (86.8, 67.1)
- added R415: 100Ω, PCM_JLCPCB:R_0402, F.Cu at (86.8, 72.7)
- added R416: 10kΩ, PCM_JLCPCB:R_0402, F.Cu at (90.2, 71.9)
- added R417: 100Ω, PCM_JLCPCB:R_0402, F.Cu at (90.2, 72.7)
- added R418: 0Ω, PCM_JLCPCB:R_0402, F.Cu at (90.2, 67.1)
- added R419: 10kΩ, PCM_JLCPCB:R_0402, F.Cu at (93.6, 71.9)
- added R420: 100Ω, PCM_JLCPCB:R_0402, F.Cu at (93.6, 72.7)
- added R421: 0Ω, PCM_JLCPCB:R_0402, F.Cu at (93.6, 67.1)
- added R422: 10kΩ, PCM_JLCPCB:R_0402, F.Cu at (77.4, 69.5)
- added R423: 10kΩ, PCM_JLCPCB:R_0402, F.Cu at (80.4, 71.9)
- added R424: 10kΩ, PCM_JLCPCB:R_0402, F.Cu at (66.1, 69.5)
- added R425: 10kΩ, PCM_JLCPCB:R_0402, F.Cu at (69.1, 71.9)
- added R426: 100Ω, PCM_JLCPCB:R_0402, F.Cu at (80.4, 72.7)
- added R427: 100Ω, PCM_JLCPCB:R_0402, F.Cu at (69.1, 72.7)
- added R428: 10kΩ, PCM_JLCPCB:R_0402, F.Cu at (54.9, 69.5)
- added R429: 10kΩ, PCM_JLCPCB:R_0402, F.Cu at (57.9, 71.9)
- added R430: 100Ω, PCM_JLCPCB:R_0402, F.Cu at (57.9, 72.7)
Routing:
- net GND: track 121.2 -> 137.2 mm, vias 104 -> 113
- net /GPIO connector2/MOSFET power stage/output: track 0.00 -> 9.73 mm
- net /GPIO connector1/MOSFET power stage/output: track 0.00 -> 9.73 mm
- net /GPIO connector/MOSFET power stage/output: track 0.00 -> 9.73 mm
- net Net-(J8-Pin_2): track 0.00 -> 7.19 mm
- net /GPIO connector2/input: track 0.00 -> 5.52 mm
- net /GPIO connector1/input: track 0.00 -> 5.52 mm
- net /GPIO connector/input: track 0.00 -> 5.52 mm
- net Net-(J8-Pin_3): track 0.00 -> 4.19 mm
- net Net-(J8-Pin_4): track 0.00 -> 4.03 mm
- net Net-(Q403-G): track 0.00 -> 2.66 mm
- net Net-(Q407-G): track 0.00 -> 2.66 mm
- net Net-(Q406-G): track 0.00 -> 2.66 mm
- net Net-(Q405-G): track 0.00 -> 2.66 mm
- net Net-(Q402-G): track 0.00 -> 2.66 mm
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
Commit message: [#1] Connect LED connector to MCU
Parts:
- added F301: Fuse, PCM_JLCPCB:R_0603, F.Cu at (49.4, 62.3)
- added TP303: TestPoint, TestPoint:TestPoint_Pad_D1.0mm, F.Cu at (47.4, 61.5)
Connections:
- J10 pad 1: +12V_FUSED -> +12V_GPIO
- J11 pad 1: +12V_FUSED -> +12V_GPIO
- J9 pad 1: +12V_FUSED -> +12V_GPIO
- R413 pad 1: /RGB LED connector/G -> /MCU/EXT_LED_G
- R415 pad 1: /RGB LED connector/G -> /MCU/EXT_LED_G
- R416 pad 1: /RGB LED connector/R -> /MCU/EXT_LED_R
- R417 pad 1: /RGB LED connector/R -> /MCU/EXT_LED_R
- R419 pad 1: /RGB LED connector/B -> /MCU/EXT_LED_B
- R420 pad 1: /RGB LED connector/B -> /MCU/EXT_LED_B
- U403 pad 15: unconnected-(U403-PC0-Pad15) -> /MCU/EXT_LED_B
- U403 pad 16: unconnected-(U403-PC1-Pad16) -> /MCU/EXT_LED_R
- U403 pad 17: unconnected-(U403-PC2-Pad17) -> /MCU/EXT_LED_G
Routing:
- net /MCU/EXT_LED_G: track 0.00 -> 54.7 mm, vias 0 -> 2
- net /MCU/EXT_LED_R: track 0.00 -> 48.3 mm, vias 0 -> 2
- net /MCU/EXT_LED_B: track 0.00 -> 47.9 mm, vias 0 -> 2
- net +12V_GPIO: track 0.00 -> 2.00 mm
- net /RGB LED connector/G: track 1.33 -> 0.00 mm
- net /RGB LED connector/R: track 1.33 -> 0.00 mm
- net /RGB LED connector/B: track 1.33 -> 0.00 mm
- added copper zone on F.Cu, net +12V_GPIO

Commit message: [#1] Connect all GPIO connectors to MCU
Connections:
- net /GPIO connector/MOSFET power stage/output renamed /GPIO connector 0/MOSFET power stage/output
- net /GPIO connector1/MOSFET power stage/output renamed /GPIO connector 1/MOSFET power stage/output
- net /GPIO connector2/MOSFET power stage/output renamed /GPIO connector 2/MOSFET power stage/output
- J10 pad 3: /GPIO connector1/input -> /GPIO connector 1/input
- J11 pad 3: /GPIO connector2/input -> /GPIO connector 2/input
- J9 pad 3: /GPIO connector/input -> /GPIO connector 0/input
- R422 pad 1: /GPIO connector/input -> /GPIO connector 0/input
- R423 pad 1: /GPIO connector/output -> /GPIO connector 0/output
- R424 pad 1: /GPIO connector1/input -> /GPIO connector 1/input
- R425 pad 1: /GPIO connector1/output -> /GPIO connector 1/output
- R426 pad 1: /GPIO connector/output -> /GPIO connector 0/output
- R427 pad 1: /GPIO connector1/output -> /GPIO connector 1/output
- R428 pad 1: /GPIO connector2/input -> /GPIO connector 2/input
- R429 pad 1: /GPIO connector2/output -> /GPIO connector 2/output
- R430 pad 1: /GPIO connector2/output -> /GPIO connector 2/output
- U403 pad 18: unconnected-(U403-PC3-Pad18) -> /GPIO connector 0/output
- U403 pad 23: unconnected-(U403-PA0-Pad23) -> /GPIO connector 0/input
- U403 pad 24: unconnected-(U403-PA1-Pad24) -> /GPIO connector 1/output
- U403 pad 25: unconnected-(U403-PA2-Pad25) -> /GPIO connector 1/input
- U403 pad 26: unconnected-(U403-PA3-Pad26) -> /GPIO connector 2/output
- U403 pad 29: unconnected-(U403-PA4-Pad29) -> /GPIO connector 2/input
Routing:
- net /GPIO connector 2/input: track 0.00 -> 87.8 mm, vias 0 -> 2
- net /GPIO connector 2/output: track 0.00 -> 74.0 mm, vias 0 -> 2
- net /GPIO connector 1/input: track 0.00 -> 72.9 mm, vias 0 -> 2
- net /GPIO connector 0/input: track 0.00 -> 67.2 mm, vias 0 -> 2
- net /GPIO connector 1/output: track 0.00 -> 63.1 mm, vias 0 -> 2
- net /GPIO connector 0/output: track 0.00 -> 57.7 mm, vias 0 -> 2
- net /GPIO connector2/input: track 5.52 -> 0.00 mm
- net /GPIO connector1/input: track 5.52 -> 0.00 mm
- net /GPIO connector/input: track 5.52 -> 0.00 mm
- net /MCU/EXT_LED_G: track 54.7 -> 53.2 mm
- net /GPIO connector2/output: track 1.33 -> 0.00 mm
- net /GPIO connector1/output: track 1.33 -> 0.00 mm
- net /GPIO connector/output: track 1.33 -> 0.00 mm
- net /MCU/EXT_LED_R: track 48.3 -> 47.6 mm

Commit message: [#1] Connect GPIOR to MCU
Connections:
- U403 pad 30: unconnected-(U403-PA5-Pad30) -> /Backplane/GPIOR15
- U403 pad 31: unconnected-(U403-PA6-Pad31) -> /Backplane/GPIOR14
- U403 pad 32: unconnected-(U403-PA7-Pad32) -> /Backplane/GPIOR13
- U403 pad 33: unconnected-(U403-PC4-Pad33) -> /Backplane/GPIOR12
- U403 pad 34: unconnected-(U403-PC5-Pad34) -> /Backplane/GPIOR11
- U403 pad 35: unconnected-(U403-PB0-Pad35) -> /Backplane/GPIOR10
- U403 pad 36: unconnected-(U403-PB1-Pad36) -> /Backplane/GPIOR9
- U403 pad 38: unconnected-(U403-PE7-Pad38) -> /Backplane/GPIOR8
- U403 pad 39: unconnected-(U403-PE8-Pad39) -> /Backplane/GPIOR7
- U403 pad 40: unconnected-(U403-PE9-Pad40) -> /Backplane/GPIOR6
- U403 pad 41: unconnected-(U403-PE10-Pad41) -> /Backplane/GPIOR5
- U403 pad 42: unconnected-(U403-PE11-Pad42) -> /Backplane/GPIOR4
- U403 pad 43: unconnected-(U403-PE12-Pad43) -> /Backplane/GPIOR3
- U403 pad 44: unconnected-(U403-PE13-Pad44) -> /Backplane/GPIOR2
- U403 pad 45: unconnected-(U403-PE14-Pad45) -> /Backplane/GPIOR1
- U403 pad 46: unconnected-(U403-PE15-Pad46) -> /Backplane/GPIOR0
Routing:
- net /Backplane/GPIOR15: track 0.00 -> 66.3 mm, vias 0 -> 1
- net /Backplane/GPIOR14: track 0.00 -> 63.5 mm, vias 0 -> 1
- net /Backplane/GPIOR13: track 0.00 -> 61.5 mm, vias 0 -> 1
- net /Backplane/GPIOR12: track 0.00 -> 58.0 mm, vias 0 -> 1
- net /Backplane/GPIOR11: track 0.00 -> 54.6 mm, vias 0 -> 1
- net /Backplane/GPIOR10: track 0.00 -> 52.5 mm, vias 0 -> 1
- net /Backplane/GPIOR9: track 0.00 -> 49.2 mm, vias 0 -> 1
- net /Backplane/GPIOR8: track 0.00 -> 46.7 mm, vias 0 -> 1
- net /Backplane/GPIOR7: track 0.00 -> 43.7 mm, vias 0 -> 1
- net /Backplane/GPIOR6: track 0.00 -> 42.3 mm, vias 0 -> 1
- net /Backplane/GPIOR5: track 0.00 -> 39.2 mm, vias 0 -> 1
- net /Backplane/GPIOR4: track 0.00 -> 38.1 mm, vias 0 -> 1
- net /Backplane/GPIOR3: track 0.00 -> 35.4 mm, vias 0 -> 1
- net /Backplane/GPIOR2: track 0.00 -> 34.7 mm, vias 0 -> 1
- net /Backplane/GPIOR1: track 0.00 -> 32.5 mm, vias 0 -> 1
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