File: gpio-module.kicad_pcb (KiCad board)
At the start: 4 copper layers, 100 x 100 mm, 196 parts, among them J10 Molex_Micro-Fit_3.0 2x2, J11 Molex_Micro-Fit_3.0 2x2, J200 09031967921, J8 Molex_Micro-Fit_3.0 2x2, J800 USB_C_Receptacle_USB2.0_16P, J9 Molex_Micro-Fit_3.0 2x2, Q401 AO3400A, Q402 AO3400A, Q403 AO3400A, Q405 AO3400A, Q406 AO3400A, Q407 AO3400A, Q700 MMST3904, U100 W25Q128, U300 TPS563200, U301 TPS563200, U302 CH334P, U401 TPD2E2U06DCK, U402 TPD2E2U06DCK, U403 STM32H562VGTx, U500 TJA1044GTK_3Z, U600 TJA1044GTK_3Z, U700 STM32F103CBTx, U801 FSUSB42UMX, X300 Q13FC1350000400, Y400 ASE-xxxMHz, Y700 Crystal_GND24, Y900 Crystal_GND24

Commit message: [#1] Connect 12V to front connectors, connect GPIOL to MCU
Parts:
- moved TP303 3.51 mm to (50.4, 63.3)
- moved F301 1.20 mm to (48.2, 62.2)
Connections:
- U403 pad 53: unconnected-(U403-PB14-Pad53) -> /Backplane/GPIOL15
- U403 pad 54: unconnected-(U403-PB15-Pad54) -> /Backplane/GPIOL14
- U403 pad 55: unconnected-(U403-PD8-Pad55) -> /Backplane/GPIOL13
- U403 pad 56: unconnected-(U403-PD9-Pad56) -> /Backplane/GPIOL12
- U403 pad 57: unconnected-(U403-PD10-Pad57) -> /Backplane/GPIOL11
- U403 pad 61: unconnected-(U403-PD14-Pad61) -> /Backplane/GPIOL10
- U403 pad 62: unconnected-(U403-PD15-Pad62) -> /Backplane/GPIOL9
- U403 pad 63: unconnected-(U403-PC6-Pad63) -> /Backplane/GPIOL8
- U403 pad 64: unconnected-(U403-PC7-Pad64) -> /Backplane/GPIOL7
- U403 pad 65: unconnected-(U403-PC8-Pad65) -> /Backplane/GPIOL6
- U403 pad 66: unconnected-(U403-PC9-Pad66) -> /Backplane/GPIOL5
- U403 pad 67: unconnected-(U403-PA8-Pad67) -> /Backplane/GPIOL4
- U403 pad 68: unconnected-(U403-PA9-Pad68) -> /Backplane/GPIOL3
- U403 pad 69: unconnected-(U403-PA10-Pad69) -> /Backplane/GPIOL2
- U403 pad 78: unconnected-(U403-PC10-Pad78) -> /Backplane/GPIOL1
- U403 pad 79: unconnected-(U403-PC11-Pad79) -> /Backplane/GPIOL0
Routing:
- net /Backplane/GPIOL15: track 0.00 -> 71.5 mm, vias 0 -> 1
- net /Backplane/GPIOL14: track 0.00 -> 68.0 mm, vias 0 -> 1
- net /Backplane/GPIOL13: track 0.00 -> 66.7 mm, vias 0 -> 1
- net /Backplane/GPIOL12: track 0.00 -> 63.8 mm, vias 0 -> 1
- net /Backplane/GPIOL11: track 0.00 -> 62.4 mm, vias 0 -> 1
- net /Backplane/GPIOL10: track 0.00 -> 60.2 mm, vias 0 -> 1
- net /Backplane/GPIOL9: track 0.00 -> 58.8 mm, vias 0 -> 1
- net /Backplane/GPIOL8: track 0.00 -> 55.8 mm, vias 0 -> 1
- net /Backplane/GPIOL7: track 0.00 -> 54.6 mm, vias 0 -> 1
- net /Backplane/GPIOL6: track 0.00 -> 51.8 mm, vias 0 -> 1
- net /Backplane/GPIOL5: track 0.00 -> 50.6 mm, vias 0 -> 1
- net /Backplane/GPIOL1: track 0.00 -> 47.6 mm, vias 0 -> 1
- net /Backplane/GPIOL4: track 0.00 -> 47.4 mm, vias 0 -> 1
- net /Backplane/GPIOL3: track 0.00 -> 46.9 mm, vias 0 -> 1
- net /Backplane/GPIOL0: track 0.00 -> 46.9 mm, vias 0 -> 1
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
Commit message: [#1] Improve GPIO tracks spacing
Routing:
- net GND: track 137.2 -> 108.4 mm, vias 94 -> 89
- net /Backplane/GPIOL15: track 71.5 -> 74.2 mm
- net /Backplane/GPIOL14: track 68.0 -> 70.4 mm
- net /Backplane/GPIOL13: track 66.7 -> 68.6 mm
- net /Backplane/GPIOL12: track 63.8 -> 65.2 mm
- net /Backplane/GPIOL9: track 58.8 -> 60.0 mm
- net /Backplane/GPIOL11: track 62.4 -> 63.5 mm
- net /Backplane/GPIOL10: track 60.2 -> 61.3 mm
- net /Backplane/GPIOL8: track 55.8 -> 56.7 mm
- net /MCU/EXT_LED_G: track 53.2 -> 52.6 mm
- net /Backplane/GPIOL7: track 54.6 -> 55.2 mm
- net /GPIO connector 2/input: track 88.0 -> 88.5 mm
- net /Backplane/GPIOL0: track 46.9 -> 46.4 mm

Commit message: [#1] Connect power to the RGB LED connector, minor tracks corrections
Parts:
- added kibuzzard-682A47D8: G***, kibuzzard-682A47D8, F.Cu at (50.4, 67.2)
- moved F301 3.00 mm to (45.2, 62.2)
Routing:
- net +5V: track 38.2 -> 130.6 mm
- net /MCU/USR_BUTTON: track 108.2 -> 106.8 mm
- net /MCU/EXT_LED_G: track 52.6 -> 52.1 mm

Commit message: [#1] Add connectors descriptions on silkscreen
Other:
- board text added: "12V LOAD"
- board text added: "A C_{B}"
- board text added: "BUTTON"
- board text added: "C_{G} C_{R}"
- board text added: "GPIO 0"
- board text added: "GPIO 1"
- board text added: "GPIO 2"
- board text added: "RGB LED"

Commit message: [#1] Clear ERC and DRC
Routing:
- net /Backplane/GPIOL10: track 61.3 -> 64.4 mm
- net /Backplane/GPIOL9: track 60.0 -> 59.4 mm
