File: gpio-module.kicad_pcb (KiCad board)
At the start: 4 copper layers, 100 x 100 mm, 197 parts, among them J10 Molex_Micro-Fit_3.0 2x2, J11 Molex_Micro-Fit_3.0 2x2, J200 09031967921, J8 Molex_Micro-Fit_3.0 2x2, J800 USB_C_Receptacle_USB2.0_16P, J9 Molex_Micro-Fit_3.0 2x2, Q401 AO3400A, Q402 AO3400A, Q403 AO3400A, Q405 AO3400A, Q406 AO3400A, Q407 AO3400A, Q700 MMST3904, U100 W25Q128, U300 TPS563200, U301 TPS563200, U302 CH334P, U401 TPD2E2U06DCK, U402 TPD2E2U06DCK, U403 STM32H562VGTx, U500 TJA1044GTK_3Z, U600 TJA1044GTK_3Z, U700 STM32F103CBTx, U801 FSUSB42UMX, X300 Q13FC1350000400, Y400 ASE-xxxMHz, Y700 Crystal_GND24, Y900 Crystal_GND24

Commit message: [#1] Add voltage divider to GPIO input
Parts:
- added R431: 1kΩ, PCM_JLCPCB:R_0402, F.Cu at (77.4, 68.5)
- added R432: 1kΩ, PCM_JLCPCB:R_0402, F.Cu at (66.1, 68.5)
- added R433: 1kΩ, PCM_JLCPCB:R_0402, F.Cu at (54.9, 68.5)
- moved R422 1.00 mm to (77.4, 70.5)
- moved R424 1.00 mm to (66.1, 70.5)
- moved R428 1.00 mm to (54.9, 70.5)
Connections:
- J10 pad 3: /GPIO connector 1/input -> Net-(J10-Pin_3)
- J11 pad 3: /GPIO connector 2/input -> Net-(J11-Pin_3)
- J9 pad 3: /GPIO connector 0/input -> Net-(J9-Pin_3)
Routing:
- net /GPIO connector 0/input: track 67.2 -> 61.7 mm
- net /GPIO connector 2/input: track 88.5 -> 83.0 mm
- net /GPIO connector 1/input: track 72.9 -> 67.5 mm
- net Net-(J9-Pin_3): track 0.00 -> 4.52 mm
- net Net-(J11-Pin_3): track 0.00 -> 4.52 mm
- net Net-(J10-Pin_3): track 0.00 -> 4.52 mm

Commit message: change RGB to CH3 and change pinout
Parts:
- removed Q401, Q402, Q403: AO3400A, PCM_JLCPCB:Q_SOT-23
- removed R413, R416, R419: 10kΩ, PCM_JLCPCB:R_0402
- removed R414, R418: 0Ω, PCM_JLCPCB:R_0402
- removed R415, R417, R420: 100Ω, PCM_JLCPCB:R_0402
- removed R431, R432, R433: 1kΩ, PCM_JLCPCB:R_0402
- added Q408: AO3400A, PCM_JLCPCB:Q_SOT-23, F.Cu at (91.7, 69.5)
- added R434: 1kΩ, PCM_JLCPCB:R_0402, F.Cu at (77.4, 68.5)
- added R435: 10kΩ, PCM_JLCPCB:R_0402, F.Cu at (88.7, 70.4)
- added R436: 10kΩ, PCM_JLCPCB:R_0402, F.Cu at (91.7, 71.9)
- added R437: 100Ω, PCM_JLCPCB:R_0402, F.Cu at (91.7, 72.7)
- added R438: 1kΩ, PCM_JLCPCB:R_0402, F.Cu at (66.1, 68.5)
- added R439: 1kΩ, PCM_JLCPCB:R_0402, F.Cu at (88.7, 68.5)
- R421: value 0Ω -> 1kΩ
- moved R421 38.7 mm to (54.9, 68.5), turned to -90 degrees
- moved R424 0.05 mm to (66.1, 70.5)
Connections:
- J10 pad 4: +3V3 -> +5V
- J11 pad 4: +3V3 -> +5V
- J8 pad 1: +5V -> +12V_GPIO
- J8 pad 2: Net-(J8-Pin_2) -> /GPIO connector 3/MOSFET power stage/output
- J8 pad 4: Net-(J8-Pin_4) -> +5V
- J9 pad 4: +3V3 -> +5V
- R421 pad 1: Net-(J8-Pin_2) -> Net-(J11-Pin_3)
- R421 pad 2: /RGB LED connector/MOSFET power stage2/output -> /GPIO connector 2/input
- U403 pad 15: /MCU/EXT_LED_B -> unconnected-(U403-PC0-Pad15)
- U403 pad 16: /MCU/EXT_LED_R -> /GPIO connector 3/input
- U403 pad 17: /MCU/EXT_LED_G -> /GPIO connector 3/output
Routing:
- net /MCU/EXT_LED_G: track 52.1 -> 0.00 mm, vias 2 -> 0
- net /GPIO connector 3/input: track 0.00 -> 51.0 mm, vias 0 -> 2
- net /GPIO connector 3/output: track 0.00 -> 47.8 mm, vias 0 -> 2
- net /MCU/EXT_LED_B: track 47.4 -> 0.00 mm, vias 2 -> 0
- net /MCU/EXT_LED_R: track 47.4 -> 0.00 mm, vias 2 -> 0
- net +5V: track 130.6 -> 173.2 mm
- net /GPIO connector 3/MOSFET power stage/output: track 0.00 -> 9.23 mm
- net Net-(J8-Pin_2): track 7.19 -> 0.00 mm
- net Net-(J8-Pin_3): track 4.19 -> 0.00 mm
- net Net-(J8-Pin_4): track 4.03 -> 0.00 mm
- net GND: track 108.4 -> 105.7 mm, vias 89 -> 88
- net Net-(Q403-G): track 2.66 -> 0.00 mm
- net Net-(Q402-G): track 2.66 -> 0.00 mm
- net Net-(Q401-G): track 2.66 -> 0.00 mm
- net Net-(Q408-G): track 0.00 -> 2.55 mm
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Other:
- board text added: "12V"
- board text added: "12V FUSE"
- board text added: "5V"
- board text added: "CH0"
- board text added: "CH1"
- board text added: "CH2"
- board text added: "CH3"
- board text added: "F PANEL"
- board text added: "GPIO"
- board text removed: "12V LOAD"
- board text removed: "A C_{B}"
- board text removed: "BUTTON"
- board text removed: "C_{G} C_{R}"
- board text removed: "GPIO 0"
- board text removed: "GPIO 1"
- board text removed: "GPIO 2"
- board text removed: "RGB LED"

Commit message: fix git sync issue
Routing:
- net +5V: track 173.2 -> 168.5 mm, vias 10 -> 14
- net Net-(J8-Pin_3): track 0.00 -> 4.51 mm
- net /GPIO connector 3/input: track 51.0 -> 51.9 mm
Other:
- board text added: "MAIN MODULE"
