File: mcu.kicad_sch (KiCad schematic)
At the start: 39 parts, among them U403 STM32H562VGTx, X300 Q13FC1350000400, Y400 ASE-xxxMHz

Commit message: [#1] Init project from base-module template
Other:
- title: ModuCard BM STM32H562VGT6 -> ModuCard GPIO module
Changed lines of the file:
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@@
 	(paper "A4")
 	(title_block
-		(title "ModuCard BM STM32H562VGT6")
-		(date "2025-04-18")
-		(rev "1.1.0")
+		(title "ModuCard GPIO module")
+		(date "2025-04-19")
+		(rev "1.0.0")
 		(company "KoNaR")
 		(comment 1 "Base project authors: Dominik Pluta, Artem Horiunov")
-		(comment 2 "Project author: <author>")
+		(comment 2 "Project author: Dominik Pluta")
 	)

Commit message: [#1] Connect LED connector to MCU
Connections:
- net EXT_LED_B: now reaches U403.15 (PC0)
- net EXT_LED_R: now reaches U403.16 (PC1)
- net EXT_LED_G: now reaches U403.17 (PC2)
- no-connect marks 58 -> 54

Commit message: [#1] Connect all GPIO connectors to MCU
Connections:
- net GPIO_0_OUT: now reaches U403.18 (PC3)
- net GPIO_0_IN: now reaches U403.23 (PA0)
- net GPIO_1_OUT: now reaches U403.24 (PA1)
- net GPIO_1_IN: now reaches U403.25 (PA2)
- net GPIO_2_OUT: now reaches U403.26 (PA3)
- net GPIO_2_IN: now reaches U403.29 (PA4)
- no-connect marks 54 -> 49

Commit message: [#1] Connect GPIOR to MCU
Connections:
- net GPIOR15: now reaches U403.30 (PA5)
- net GPIOR14: now reaches U403.31 (PA6)
- net GPIOR13: now reaches U403.32 (PA7)
- net GPIOR12: now reaches U403.33 (PC4)
- net GPIOR11: now reaches U403.34 (PC5)
- net GPIOR10: now reaches U403.35 (PB0)
- net GPIOR9: now reaches U403.36 (PB1)
- net GPIOR8: now reaches U403.38 (PE7)
- net GPIOR7: now reaches U403.39 (PE8)
- net GPIOR6: now reaches U403.40 (PE9)
- net GPIOR5: now reaches U403.41 (PE10)
- net GPIOR4: now reaches U403.42 (PE11)
- net GPIOR3: now reaches U403.43 (PE12)
- net GPIOR2: now reaches U403.44 (PE13)
- net GPIOR1: now reaches U403.45 (PE14)
- net GPIOR0: now reaches U403.46 (PE15)
- no-connect marks 49 -> 33

Commit message: [#1] Connect 12V to front connectors, connect GPIOL to MCU
Connections:
- net GPIOL0: now also U403.79 (PC11)
- net GPIOL1: now also U403.78 (PC10)
- net GPIOL10: now also U403.61 (PD14)
- net GPIOL11: now also U403.57 (PD10)
- net GPIOL12: now also U403.56 (PD9)
- net GPIOL13: now also U403.55 (PD8)
- net GPIOL14: now also U403.54 (PB15)
- net GPIOL15: now also U403.53 (PB14)
- net GPIOL2: now also U403.69 (PA10)
- net GPIOL3: now also U403.68 (PA9)
- net GPIOL4: now also U403.67 (PA8)
- net GPIOL5: now also U403.66 (PC9)
- net GPIOL6: now also U403.65 (PC8)
- net GPIOL7: now also U403.64 (PC7)
- net GPIOL8: now also U403.63 (PC6)
- net GPIOL9: now also U403.62 (PD15)
- no-connect marks 33 -> 17
