File: mcu.kicad_sch (KiCad schematic)
At the start: 39 parts, among them U403 STM32H562VGTx, X300 Q13FC1350000400, Y400 ASE-xxxMHz

Commit message: Replace RGB with CH3 and adjust silk
Connections:
- net EXT_LED_B: no longer names the net of U403.15 (PC0)
- net EXT_LED_G renamed GPIO_3_OUT
- net EXT_LED_R renamed GPIO_3_IN
- no-connect marks 17 -> 18
