File: mcu.kicad_sch (KiCad schematic)
At the start: 39 parts, among them U403 STM32H562VGTx, X300 Q13FC1350000400, Y400 ASE-xxxMHz

Commit message: [#8] Fix LEDs resistors values
Parts:
- removed R400: 1.2kΩ, PCM_JLCPCB:R_0402, symbol PCM_JLCPCB-Resistors:0402,1.2kΩ
- removed R408: 220Ω, PCM_JLCPCB:R_0402, symbol PCM_JLCPCB-Resistors:0402,220Ω
- removed R409: 100Ω, PCM_JLCPCB:R_0402, symbol PCM_JLCPCB-Resistors:0402,100Ω
- added R414, R415, R416: 220Ω, PCM_JLCPCB:R_0402, symbol PCM_JLCPCB-Resistors:0402,220Ω
Connections:
- net +3V3: now also R414.1
- net STATUS_LED: now also R415.1
- net USER_LED_1: now also R416.1
- net at LED301.3: now also R414.2
- net at LED300.1: now also R416.2
- net at LED301.1: now also R415.2

Commit message: [#1] Fill out schematic title block, connect GPIOs on the schematic
Connections:
- net GPIO_3_IN: now reaches U403.16 (PC1)
- net GPIO_3_OUT: now reaches U403.17 (PC2)
- net GPIO_0_OUT: now reaches U403.18 (PC3)
- net GPIO_0_IN: now reaches U403.23 (PA0)
- net GPIO_1_OUT: now reaches U403.24 (PA1)
- net GPIO_1_IN: now reaches U403.25 (PA2)
- net GPIO_2_OUT: now reaches U403.26 (PA3)
- net GPIO_2_IN: now reaches U403.29 (PA4)
- net GPIOR15: now reaches U403.30 (PA5)
- net GPIOR14: now reaches U403.31 (PA6)
- net GPIOR13: now reaches U403.32 (PA7)
- net GPIOR12: now reaches U403.33 (PC4)
- net GPIOR11: now reaches U403.34 (PC5)
- net GPIOR10: now reaches U403.35 (PB0)
- net GPIOR9: now reaches U403.36 (PB1)
- net GPIOR8: now reaches U403.38 (PE7)
- net GPIOR7: now reaches U403.39 (PE8)
- net GPIOR6: now reaches U403.40 (PE9)
- net GPIOR5: now reaches U403.41 (PE10)
- net GPIOR4: now reaches U403.42 (PE11)
- net GPIOR3: now reaches U403.43 (PE12)
- net GPIOR2: now reaches U403.44 (PE13)
- net GPIOR1: now reaches U403.45 (PE14)
- net GPIOR0: now reaches U403.46 (PE15)
- net GPIOL15: now reaches U403.53 (PB14)
- net GPIOL14: now reaches U403.54 (PB15)
- net GPIOL13: now reaches U403.55 (PD8)
- net GPIOL12: now reaches U403.56 (PD9)
- net GPIOL11: now reaches U403.57 (PD10)
- net GPIOL10: now reaches U403.61 (PD14)
- net GPIOL9: now reaches U403.62 (PD15)
- net GPIOL8: now reaches U403.63 (PC6)
- net GPIOL7: now reaches U403.64 (PC7)
- net GPIOL6: now reaches U403.65 (PC8)
- net GPIOL5: now reaches U403.66 (PC9)
- net GPIOL4: now reaches U403.67 (PA8)
- net GPIOL3: now reaches U403.68 (PA9)
- net GPIOL2: now reaches U403.69 (PA10)
- net GPIOL1: now reaches U403.78 (PC10)
- net GPIOL0: now reaches U403.79 (PC11)
- no-connect marks 58 -> 18
Other:
- note added: "BACKPLANE GPIO"
- title: ModuCard BM STM32H562VGT6 -> ModuCard GPIO module
- moved on the sheet: C313, C314, C423, C424, C425, C426, C432, FB401, LED300A, LED300B, LED301A, LED301B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
Changed lines of the file:
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@@
 	(generator "eeschema")
 	(generator_version "9.0")
-	(paper "A4")
+	(paper "A3")
 	(title_block
-		(title "ModuCard BM STM32H562VGT6")
-		(date "2025-04-18")
-		(rev "1.1.1")
+		(title "ModuCard GPIO module")
+		(date "2025-06-19")
+		(rev "1.0.0")
 		(company "KoNaR")
 		(comment 1 "Base project authors: Dominik Pluta, Artem Horiunov")
-		(comment 2 "Project author: <author>")
+		(comment 2 "Project author: Dominik Pluta")
 	)

Commit message: [#6] Define ADC pins, start rerouting
Connections:
- net GPIO_0_IN: now also U403.16 (PC1); no longer U403.23 (PA0)
- net GPIO_0_OUT: no longer U403.18 (PC3)
- net GPIO_1_IN: now also U403.17 (PC2); no longer U403.25 (PA2)
- net GPIO_2_IN: now also U403.18 (PC3); no longer U403.29 (PA4)
- net GPIO_3_IN: now also U403.15 (PC0); no longer U403.16 (PC1)
- net GPIO_3_OUT: no longer U403.17 (PC2)
- no-connect marks 18 -> 17

Commit message: [#6] WIP: connect GPIO
Connections:
- net GPIO_0_OUT: now also U403.87 (PD6)
- net GPIO_1_OUT: now also U403.86 (PD5); no longer U403.24 (PA1)
- net GPIO_2_OUT: now also U403.85 (PD4); no longer U403.26 (PA3)
- net GPIO_3_OUT: now also U403.88 (PD7)
- no-connect marks 17 -> 13
