File: gpio-connector.kicad_sch (KiCad schematic)
At the start: 3 parts, among them J9 Molex_Micro-Fit_3.0 2x2

Commit message: change RGB to CH3 and change pinout
Parts:
- renumbered R431 to R
Connections:
- net +3V3 renamed +5V
Changed lines of the file:
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@@
 	)
 	(hierarchical_label "input"
-		(shape input)
+		(shape output)
 		(at 120.65 96.52 180)
 		(effects
@@
 		(on_board yes)
 		(dnp no)
-		(property "Reference" "R431"
+		(property "Reference" "R"
 			(at 179.07 88.9 0)
 			(effects
@@
 		)
 		(instances
-			(project ""
-				(path "/090a8e41-87a8-4fb1-998b-60a2c0dc4cee/5f7db16d-834d-414e-a24b-79c654644ccf"
-					(reference "R431")
-					(unit 1)
-				)
-				(path "/090a8e41-87a8-4fb1-998b-60a2c0dc4cee/83bb9cd3-e66c-42fc-8ebd-53e27e95abe3"
-					(reference "R432")
-					(unit 1)
-				)
-				(path "/090a8e41-87a8-4fb1-998b-60a2c0dc4cee/b4df952d-7669-4a91-8ac9-9d4461ce2e59"
-					(reference "R433")
+			(project "gpio-module"
+				(path "/090a8e41-87a8-4fb1-998b-60a2c0dc4cee/a33dc8b1-4620-4cf7-8065-8ae8af0e84cf"
+					(reference "R434")
 					(unit 1)
 				)
@@
 					(unit 1)
 				)
+				(path "/090a8e41-87a8-4fb1-998b-60a2c0dc4cee/a33dc8b1-4620-4cf7-8065-8ae8af0e84cf"
+					(reference "#PWR0489")
+					(unit 1)
+				)
 				(path "/090a8e41-87a8-4fb1-998b-60a2c0dc4cee/b4df952d-7669-4a91-8ac9-9d4461ce2e59"
 					(reference "#PWR0482")
@@
 					(unit 1)
 				)
+				(path "/090a8e41-87a8-4fb1-998b-60a2c0dc4cee/a33dc8b1-4620-4cf7-8065-8ae8af0e84cf"
+					(reference "R435")
+					(unit 1)
+				)
 				(path "/090a8e41-87a8-4fb1-998b-60a2c0dc4cee/b4df952d-7669-4a91-8ac9-9d4461ce2e59"
 					(reference "R428")
@@
 					(unit 1)
 				)
+				(path "/090a8e41-87a8-4fb1-998b-60a2c0dc4cee/a33dc8b1-4620-4cf7-8065-8ae8af0e84cf"
+					(reference "#PWR0324")
+					(unit 1)
+				)
 				(path "/090a8e41-87a8-4fb1-998b-60a2c0dc4cee/b4df952d-7669-4a91-8ac9-9d4461ce2e59"
 					(reference "#PWR0313")
@@
 					(unit 1)
 				)
+				(path "/090a8e41-87a8-4fb1-998b-60a2c0dc4cee/a33dc8b1-4620-4cf7-8065-8ae8af0e84cf"
+					(reference "J8")
+					(unit 1)
+				)
 				(path "/090a8e41-87a8-4fb1-998b-60a2c0dc4cee/b4df952d-7669-4a91-8ac9-9d4461ce2e59"
 					(reference "J11")
@@
 		(on_board yes)
 		(dnp no)
-		(property "Reference" "#PWR0325"
+		(fields_autoplaced yes)
+		(property "Reference" "#PWR"
 			(at 177.8 77.47 0)
 			(effects
@@
 			)
 		)
-		(property "Value" "+3V3"
-			(at 177.8 69.85 0)
+		(property "Value" "+5V"
+			(at 177.8 68.58 0)
 			(effects
 				(font
@@
 		(instances
 			(project "gpio-module"
-				(path "/090a8e41-87a8-4fb1-998b-60a2c0dc4cee/5f7db16d-834d-414e-a24b-79c654644ccf"
-					(reference "#PWR0325")
-					(unit 1)
-				)
-				(path "/090a8e41-87a8-4fb1-998b-60a2c0dc4cee/83bb9cd3-e66c-42fc-8ebd-53e27e95abe3"
-					(reference "#PWR0326")
-					(unit 1)
-				)
-				(path "/090a8e41-87a8-4fb1-998b-60a2c0dc4cee/b4df952d-7669-4a91-8ac9-9d4461ce2e59"
-					(reference "#PWR0333")
+				(path "/090a8e41-87a8-4fb1-998b-60a2c0dc4cee/a33dc8b1-4620-4cf7-8065-8ae8af0e84cf"
+					(reference "#PWR0488")
 					(unit 1)
 				)
@@
 					(page "20")
 				)
-			)
+				(path "/090a8e41-87a8-4fb1-998b-60a2c0dc4cee/a33dc8b1-4620-4cf7-8065-8ae8af0e84cf"
+					(page "22")
+				)
+			)
