File: gpio-connector.kicad_sch (KiCad schematic)
At the start: 2 parts, among them J9 Molex_Micro-Fit_3.0 2x2

Commit message: [#1] Connect LED connector to MCU
Connections:
- net +12V_FUSED renamed +12V_GPIO
Changed lines of the file:
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@@
 			)
 		)
-		(property "Value" "+12V_FUSED"
+		(property "Value" "+12V_GPIO"
 			(at 149.86 69.85 0)
 			(effects

Commit message: [#1] Clear ERC and DRC
Changed lines of the file:
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@@
-	)
-	(symbol
-		(lib_id "power:+5V")
-		(at 287.02 110.49 0)
-		(unit 1)
-		(exclude_from_sim no)
-		(in_bom yes)
-		(on_board yes)
-		(dnp no)
-		(property "Reference" "#PWR0324"
-			(at 287.02 114.3 0)
-			(effects
-				(font
-					(size 1.27 1.27)
-				)
-				(hide yes)
-			)
-		)
-		(property "Value" "+3V3"
-			(at 287.02 106.68 0)
-			(effects
-				(font
-					(size 1.27 1.27)
-				)
-			)
-		)
-		(property "Footprint" ""
-			(at 287.02 110.49 0)
-			(effects
-				(font
-					(size 1.27 1.27)
-				)
-				(hide yes)
-			)
-		)
-		(property "Datasheet" ""
-			(at 287.02 110.49 0)
-			(effects
-				(font
-					(size 1.27 1.27)
-				)
-				(hide yes)
-			)
-		)
-		(property "Description" "Power symbol creates a global label with name \"+5V\""
-			(at 287.02 110.49 0)
-			(effects
-				(font
-					(size 1.27 1.27)
-				)
-				(hide yes)
-			)
-		)
-		(pin "1"
-		)
-		(instances
-			(project "gpio-module"
-				(path "/090a8e41-87a8-4fb1-998b-60a2c0dc4cee/5f7db16d-834d-414e-a24b-79c654644ccf"
-					(reference "#PWR0324")
-					(unit 1)
-				)
-				(path "/090a8e41-87a8-4fb1-998b-60a2c0dc4cee/83bb9cd3-e66c-42fc-8ebd-53e27e95abe3"
-					(reference "#PWR0327")
-					(unit 1)
-				)
-				(path "/090a8e41-87a8-4fb1-998b-60a2c0dc4cee/b4df952d-7669-4a91-8ac9-9d4461ce2e59"
-					(reference "#PWR0334")
-					(unit 1)
-				)
-			)
-		)
 	)
 	(symbol

Commit message: [#1] Add voltage divider to GPIO input
Parts:
- added R431: 1kΩ, PCM_JLCPCB:R_0402, symbol PCM_JLCPCB-Resistors:0402,1kΩ
Connections:
- net input: now also R431.2; no longer J9.3 (Pin_3)
- new net: J9.3 (Pin_3), R431.1

Commit message: Replace RGB with CH3 and adjust silk
Parts:
- removed R422: 10kΩ, PCM_JLCPCB:R_0402, symbol PCM_JLCPCB-Resistors:0402,10kΩ
- removed R431: 1kΩ, PCM_JLCPCB:R_0402, symbol PCM_JLCPCB-Resistors:0402,1kΩ
- added R416: 10kΩ, PCM_JLCPCB:R_0402, symbol PCM_JLCPCB-Resistors:0402,10kΩ
- added R420: 22kΩ, PCM_JLCPCB:R_0402, symbol PCM_JLCPCB-Resistors:0402,22kΩ
Connections:
- net GND: now also R420.2
- net input: now also R416.2, R420.1
- net at J9.3 (Pin_3): now also R416.1
- net +3V3 renamed +5V
