File: gpio-connector.kicad_sch (KiCad schematic)
At the start: 3 parts, among them J11 Molex_Micro-Fit_3.0 2x2

Commit message: [#1] Finish PCB
Parts:
- renumbered J11 to J9, R419 to R400, R423 to R420
Changed lines of the file:
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@@
 		(on_board yes)
 		(dnp no)
-		(property "Reference" "#PWR0482"
+		(property "Reference" "#PWR0470"
 			(at 177.8 115.57 0)
 			(effects
@@
 		(instances
 			(project "base-module"
-				(path "/090a8e41-87a8-4fb1-998b-60a2c0dc4cee/1e4742a2-145a-46a6-8222-17374fa3a593"
-					(reference "#PWR0485")
-					(unit 1)
-				)
-				(path "/090a8e41-87a8-4fb1-998b-60a2c0dc4cee/21e14c9e-8cb5-4c0d-8827-cab6b62735cd"
-					(reference "#PWR0483")
-					(unit 1)
-				)
-				(path "/090a8e41-87a8-4fb1-998b-60a2c0dc4cee/b0ae0dc1-1dc3-4071-a986-cf1be8ac718c"
-					(reference "#PWR0482")
-					(unit 1)
-				)
-				(path "/090a8e41-87a8-4fb1-998b-60a2c0dc4cee/b5a8ed9d-2492-499d-884c-f314ed804d88"
-					(reference "#PWR0484")
+				(path "/090a8e41-87a8-4fb1-998b-60a2c0dc4cee/2eacc112-c748-4514-8f19-54a63b484540"
+					(reference "#PWR0473")
+					(unit 1)
+				)
+				(path "/090a8e41-87a8-4fb1-998b-60a2c0dc4cee/3ce14170-f6f1-4e98-bfea-8e2751441f01"
+					(reference "#PWR0479")
+					(unit 1)
+				)
+				(path "/090a8e41-87a8-4fb1-998b-60a2c0dc4cee/482f7d0c-144a-4b8c-8f49-834e199b564c"
+					(reference "#PWR0470")
+					(unit 1)
+				)
+				(path "/090a8e41-87a8-4fb1-998b-60a2c0dc4cee/8f334819-7829-459d-a376-c28f1c3582e9"
+					(reference "#PWR0476")
 					(unit 1)
 				)
@@
 		(on_board yes)
 		(dnp no)
-		(property "Reference" "R419"
+		(property "Reference" "R400"
 			(at 179.324 88.9 0)
 			(effects
@@
 		(instances
 			(project "base-module"
-				(path "/090a8e41-87a8-4fb1-998b-60a2c0dc4cee/1e4742a2-145a-46a6-8222-17374fa3a593"
-					(reference "R422")
-					(unit 1)
-				)
-				(path "/090a8e41-87a8-4fb1-998b-60a2c0dc4cee/21e14c9e-8cb5-4c0d-8827-cab6b62735cd"
-					(reference "R420")
-					(unit 1)
-				)
-				(path "/090a8e41-87a8-4fb1-998b-60a2c0dc4cee/b0ae0dc1-1dc3-4071-a986-cf1be8ac718c"
+				(path "/090a8e41-87a8-4fb1-998b-60a2c0dc4cee/2eacc112-c748-4514-8f19-54a63b484540"
+					(reference "R417")
+					(unit 1)
+				)
+				(path "/090a8e41-87a8-4fb1-998b-60a2c0dc4cee/3ce14170-f6f1-4e98-bfea-8e2751441f01"
 					(reference "R419")
 					(unit 1)
 				)
-				(path "/090a8e41-87a8-4fb1-998b-60a2c0dc4cee/b5a8ed9d-2492-499d-884c-f314ed804d88"
-					(reference "R421")
+				(path "/090a8e41-87a8-4fb1-998b-60a2c0dc4cee/482f7d0c-144a-4b8c-8f49-834e199b564c"
+					(reference "R400")
+					(unit 1)
+				)
+				(path "/090a8e41-87a8-4fb1-998b-60a2c0dc4cee/8f334819-7829-459d-a376-c28f1c3582e9"
+					(reference "R418")
 					(unit 1)
 				)
@@
 		(on_board yes)
 		(dnp no)
-		(property "Reference" "#PWR0313"
+		(property "Reference" "#PWR0400"
 			(at 149.86 77.47 0)
 			(effects
@@
 		(instances
 			(project "base-module"
-				(path "/090a8e41-87a8-4fb1-998b-60a2c0dc4cee/1e4742a2-145a-46a6-8222-17374fa3a593"
-					(reference "#PWR0325")
-					(unit 1)
-				)
-				(path "/090a8e41-87a8-4fb1-998b-60a2c0dc4cee/21e14c9e-8cb5-4c0d-8827-cab6b62735cd"
-					(reference "#PWR0314")
-					(unit 1)
-				)
-				(path "/090a8e41-87a8-4fb1-998b-60a2c0dc4cee/b0ae0dc1-1dc3-4071-a986-cf1be8ac718c"
-					(reference "#PWR0313")
-					(unit 1)
-				)
-				(path "/090a8e41-87a8-4fb1-998b-60a2c0dc4cee/b5a8ed9d-2492-499d-884c-f314ed804d88"
-					(reference "#PWR0324")
+				(path "/090a8e41-87a8-4fb1-998b-60a2c0dc4cee/2eacc112-c748-4514-8f19-54a63b484540"
+					(reference "#PWR0471")
+					(unit 1)
+				)
+				(path "/090a8e41-87a8-4fb1-998b-60a2c0dc4cee/3ce14170-f6f1-4e98-bfea-8e2751441f01"
+					(reference "#PWR0477")
+					(unit 1)
+				)
+				(path "/090a8e41-87a8-4fb1-998b-60a2c0dc4cee/482f7d0c-144a-4b8c-8f49-834e199b564c"
+					(reference "#PWR0400")
+					(unit 1)
+				)
+				(path "/090a8e41-87a8-4fb1-998b-60a2c0dc4cee/8f334819-7829-459d-a376-c28f1c3582e9"
+					(reference "#PWR0474")
 					(unit 1)
 				)
@@
 		(on_board yes)
 		(dnp no)
-		(property "Reference" "R423"
+		(property "Reference" "R420"
 			(at 179.324 102.87 0)
 			(effects
@@
 		(instances
 			(project "base-module"
-				(path "/090a8e41-87a8-4fb1-998b-60a2c0dc4cee/1e4742a2-145a-46a6-8222-17374fa3a593"
-					(reference "R426")
-					(unit 1)
-				)
-				(path "/090a8e41-87a8-4fb1-998b-60a2c0dc4cee/21e14c9e-8cb5-4c0d-8827-cab6b62735cd"
+				(path "/090a8e41-87a8-4fb1-998b-60a2c0dc4cee/2eacc112-c748-4514-8f19-54a63b484540"
+					(reference "R421")
+					(unit 1)
+				)
+				(path "/090a8e41-87a8-4fb1-998b-60a2c0dc4cee/3ce14170-f6f1-4e98-bfea-8e2751441f01"
 					(reference "R424")
 					(unit 1)
 				)
-				(path "/090a8e41-87a8-4fb1-998b-60a2c0dc4cee/b0ae0dc1-1dc3-4071-a986-cf1be8ac718c"
-					(reference "R423")
-					(unit 1)
-				)
-				(path "/090a8e41-87a8-4fb1-998b-60a2c0dc4cee/b5a8ed9d-2492-499d-884c-f314ed804d88"
-					(reference "R425")
+				(path "/090a8e41-87a8-4fb1-998b-60a2c0dc4cee/482f7d0c-144a-4b8c-8f49-834e199b564c"
+					(reference "R420")
+					(unit 1)
+				)
+				(path "/090a8e41-87a8-4fb1-998b-60a2c0dc4cee/8f334819-7829-459d-a376-c28f1c3582e9"
+					(reference "R422")
 					(unit 1)
 				)
@@
 		(on_board yes)
 		(dnp no)
-		(property "Reference" "J11"
+		(property "Reference" "J9"
 			(at 163.83 73.66 0)
 			(effects
@@
 		(instances
 			(project "base-module"
-				(path "/090a8e41-87a8-4fb1-998b-60a2c0dc4cee/1e4742a2-145a-46a6-8222-17374fa3a593"
-					(reference "J14")
-					(unit 1)
-				)
-				(path "/090a8e41-87a8-4fb1-998b-60a2c0dc4cee/21e14c9e-8cb5-4c0d-8827-cab6b62735cd"
-					(reference "J12")
-					(unit 1)
-				)
-				(path "/090a8e41-87a8-4fb1-998b-60a2c0dc4cee/b0ae0dc1-1dc3-4071-a986-cf1be8ac718c"
+				(path "/090a8e41-87a8-4fb1-998b-60a2c0dc4cee/2eacc112-c748-4514-8f19-54a63b484540"
+					(reference "J10")
+					(unit 1)
+				)
+				(path "/090a8e41-87a8-4fb1-998b-60a2c0dc4cee/3ce14170-f6f1-4e98-bfea-8e2751441f01"
+					(reference "J8")
+					(unit 1)
+				)
+				(path "/090a8e41-87a8-4fb1-998b-60a2c0dc4cee/482f7d0c-144a-4b8c-8f49-834e199b564c"
+					(reference "J9")
+					(unit 1)
+				)
+				(path "/090a8e41-87a8-4fb1-998b-60a2c0dc4cee/8f334819-7829-459d-a376-c28f1c3582e9"
 					(reference "J11")
-					(unit 1)
-				)
-				(path "/090a8e41-87a8-4fb1-998b-60a2c0dc4cee/b5a8ed9d-2492-499d-884c-f314ed804d88"
-					(reference "J13")
 					(unit 1)
 				)
@@
 		(dnp no)
 		(fields_autoplaced yes)
-		(property "Reference" "#PWR0103"
+		(property "Reference" "#PWR0459"
 			(at 177.8 77.47 0)
 			(effects
@@
 		(instances
 			(project "base-module"
-				(path "/090a8e41-87a8-4fb1-998b-60a2c0dc4cee/1e4742a2-145a-46a6-8222-17374fa3a593"
-					(reference "#PWR0106")
-					(unit 1)
-				)
-				(path "/090a8e41-87a8-4fb1-998b-60a2c0dc4cee/21e14c9e-8cb5-4c0d-8827-cab6b62735cd"
-					(reference "#PWR0104")
-					(unit 1)
-				)
-				(path "/090a8e41-87a8-4fb1-998b-60a2c0dc4cee/b0ae0dc1-1dc3-4071-a986-cf1be8ac718c"
-					(reference "#PWR0103")
-					(unit 1)
-				)
-				(path "/090a8e41-87a8-4fb1-998b-60a2c0dc4cee/b5a8ed9d-2492-499d-884c-f314ed804d88"
-					(reference "#PWR0105")
+				(path "/090a8e41-87a8-4fb1-998b-60a2c0dc4cee/2eacc112-c748-4514-8f19-54a63b484540"
+					(reference "#PWR0472")
+					(unit 1)
+				)
+				(path "/090a8e41-87a8-4fb1-998b-60a2c0dc4cee/3ce14170-f6f1-4e98-bfea-8e2751441f01"
+					(reference "#PWR0478")
+					(unit 1)
+				)
+				(path "/090a8e41-87a8-4fb1-998b-60a2c0dc4cee/482f7d0c-144a-4b8c-8f49-834e199b564c"
+					(reference "#PWR0459")
+					(unit 1)
+				)
+				(path "/090a8e41-87a8-4fb1-998b-60a2c0dc4cee/8f334819-7829-459d-a376-c28f1c3582e9"
+					(reference "#PWR0475")
 					(unit 1)
 				)
@@
 		(instances
 			(project "base-module"
-				(path "/090a8e41-87a8-4fb1-998b-60a2c0dc4cee/b0ae0dc1-1dc3-4071-a986-cf1be8ac718c"
+				(path "/090a8e41-87a8-4fb1-998b-60a2c0dc4cee/482f7d0c-144a-4b8c-8f49-834e199b564c"
 					(page "12")
 				)
-				(path "/090a8e41-87a8-4fb1-998b-60a2c0dc4cee/21e14c9e-8cb5-4c0d-8827-cab6b62735cd"
+				(path "/090a8e41-87a8-4fb1-998b-60a2c0dc4cee/2eacc112-c748-4514-8f19-54a63b484540"
 					(page "14")
 				)
-				(path "/090a8e41-87a8-4fb1-998b-60a2c0dc4cee/b5a8ed9d-2492-499d-884c-f314ed804d88"
+				(path "/090a8e41-87a8-4fb1-998b-60a2c0dc4cee/8f334819-7829-459d-a376-c28f1c3582e9"
 					(page "16")
 				)
-				(path "/090a8e41-87a8-4fb1-998b-60a2c0dc4cee/1e4742a2-145a-46a6-8222-17374fa3a593"
+				(path "/090a8e41-87a8-4fb1-998b-60a2c0dc4cee/3ce14170-f6f1-4e98-bfea-8e2751441f01"
 					(page "18")
 				)
