File: mosfet-power-stage.kicad_sch (KiCad schematic)
At the start: 3 parts, among them Q401 AO3400A

Commit message: Replace RGB with CH3 and adjust silk
Parts:
- renumbered Q401 to Q405, R413 to R423, R415 to R426
Changed lines of the file:
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@@
 		(on_board yes)
 		(dnp no)
-		(property "Reference" "R413"
+		(property "Reference" "R423"
 			(at 129.54 104.14 0)
 			(effects
@@
 		(instances
 			(project "gpio-module"
-				(path "/090a8e41-87a8-4fb1-998b-60a2c0dc4cee/4ad8e31a-cde3-429e-898f-5d817c85a694/0230d939-768e-429e-8928-f79ac4fd3229"
-					(reference "R419")
-					(unit 1)
-				)
-				(path "/090a8e41-87a8-4fb1-998b-60a2c0dc4cee/4ad8e31a-cde3-429e-898f-5d817c85a694/05560d46-8ccc-48df-b10d-1c3a365a35b2"
-					(reference "R416")
-					(unit 1)
-				)
-				(path "/090a8e41-87a8-4fb1-998b-60a2c0dc4cee/4ad8e31a-cde3-429e-898f-5d817c85a694/3200d16b-13e4-4f35-a189-f6ee81970efa"
-					(reference "R413")
-					(unit 1)
-				)
 				(path "/090a8e41-87a8-4fb1-998b-60a2c0dc4cee/5f7db16d-834d-414e-a24b-79c654644ccf/d3e6b829-08f5-499b-8b35-220ffa9a4993"
 					(reference "R423")
@@
 				(path "/090a8e41-87a8-4fb1-998b-60a2c0dc4cee/83bb9cd3-e66c-42fc-8ebd-53e27e95abe3/d3e6b829-08f5-499b-8b35-220ffa9a4993"
 					(reference "R425")
+					(unit 1)
+				)
+				(path "/090a8e41-87a8-4fb1-998b-60a2c0dc4cee/a33dc8b1-4620-4cf7-8065-8ae8af0e84cf/d3e6b829-08f5-499b-8b35-220ffa9a4993"
+					(reference "R436")
 					(unit 1)
 				)
@@
 		(on_board yes)
 		(dnp no)
-		(property "Reference" "R415"
+		(property "Reference" "R426"
 			(at 134.62 96.774 90)
 			(effects
@@
 		(instances
 			(project "gpio-module"
-				(path "/090a8e41-87a8-4fb1-998b-60a2c0dc4cee/4ad8e31a-cde3-429e-898f-5d817c85a694/0230d939-768e-429e-8928-f79ac4fd3229"
-					(reference "R420")
-					(unit 1)
-				)
-				(path "/090a8e41-87a8-4fb1-998b-60a2c0dc4cee/4ad8e31a-cde3-429e-898f-5d817c85a694/05560d46-8ccc-48df-b10d-1c3a365a35b2"
-					(reference "R417")
-					(unit 1)
-				)
-				(path "/090a8e41-87a8-4fb1-998b-60a2c0dc4cee/4ad8e31a-cde3-429e-898f-5d817c85a694/3200d16b-13e4-4f35-a189-f6ee81970efa"
-					(reference "R415")
-					(unit 1)
-				)
 				(path "/090a8e41-87a8-4fb1-998b-60a2c0dc4cee/5f7db16d-834d-414e-a24b-79c654644ccf/d3e6b829-08f5-499b-8b35-220ffa9a4993"
 					(reference "R426")
@@
 				(path "/090a8e41-87a8-4fb1-998b-60a2c0dc4cee/83bb9cd3-e66c-42fc-8ebd-53e27e95abe3/d3e6b829-08f5-499b-8b35-220ffa9a4993"
 					(reference "R427")
+					(unit 1)
+				)
+				(path "/090a8e41-87a8-4fb1-998b-60a2c0dc4cee/a33dc8b1-4620-4cf7-8065-8ae8af0e84cf/d3e6b829-08f5-499b-8b35-220ffa9a4993"
+					(reference "R437")
 					(unit 1)
 				)
@@
 		(on_board yes)
 		(dnp no)
-		(property "Reference" "#PWR0459"
+		(property "Reference" "#PWR0480"
 			(at 148.59 116.84 0)
 			(effects
@@
 		(instances
 			(project "gpio-module"
-				(path "/090a8e41-87a8-4fb1-998b-60a2c0dc4cee/4ad8e31a-cde3-429e-898f-5d817c85a694/0230d939-768e-429e-8928-f79ac4fd3229"
-					(reference "#PWR0474")
-					(unit 1)
-				)
-				(path "/090a8e41-87a8-4fb1-998b-60a2c0dc4cee/4ad8e31a-cde3-429e-898f-5d817c85a694/05560d46-8ccc-48df-b10d-1c3a365a35b2"
-					(reference "#PWR0472")
-					(unit 1)
-				)
-				(path "/090a8e41-87a8-4fb1-998b-60a2c0dc4cee/4ad8e31a-cde3-429e-898f-5d817c85a694/3200d16b-13e4-4f35-a189-f6ee81970efa"
-					(reference "#PWR0459")
-					(unit 1)
-				)
 				(path "/090a8e41-87a8-4fb1-998b-60a2c0dc4cee/5f7db16d-834d-414e-a24b-79c654644ccf/d3e6b829-08f5-499b-8b35-220ffa9a4993"
 					(reference "#PWR0480")
@@
 				(path "/090a8e41-87a8-4fb1-998b-60a2c0dc4cee/83bb9cd3-e66c-42fc-8ebd-53e27e95abe3/d3e6b829-08f5-499b-8b35-220ffa9a4993"
 					(reference "#PWR0481")
+					(unit 1)
+				)
+				(path "/090a8e41-87a8-4fb1-998b-60a2c0dc4cee/a33dc8b1-4620-4cf7-8065-8ae8af0e84cf/d3e6b829-08f5-499b-8b35-220ffa9a4993"
+					(reference "#PWR0491")
 					(unit 1)
 				)
@@
 		(on_board yes)
 		(dnp no)
-		(property "Reference" "#PWR0470"
+		(property "Reference" "#PWR0477"
 			(at 128.27 116.84 0)
 			(effects
@@
 		(instances
 			(project "gpio-module"
-				(path "/090a8e41-87a8-4fb1-998b-60a2c0dc4cee/4ad8e31a-cde3-429e-898f-5d817c85a694/0230d939-768e-429e-8928-f79ac4fd3229"
-					(reference "#PWR0473")
-					(unit 1)
-				)
-				(path "/090a8e41-87a8-4fb1-998b-60a2c0dc4cee/4ad8e31a-cde3-429e-898f-5d817c85a694/05560d46-8ccc-48df-b10d-1c3a365a35b2"
-					(reference "#PWR0471")
-					(unit 1)
-				)
-				(path "/090a8e41-87a8-4fb1-998b-60a2c0dc4cee/4ad8e31a-cde3-429e-898f-5d817c85a694/3200d16b-13e4-4f35-a189-f6ee81970efa"
-					(reference "#PWR0470")
-					(unit 1)
-				)
 				(path "/090a8e41-87a8-4fb1-998b-60a2c0dc4cee/5f7db16d-834d-414e-a24b-79c654644ccf/d3e6b829-08f5-499b-8b35-220ffa9a4993"
 					(reference "#PWR0477")
@@
 				(path "/090a8e41-87a8-4fb1-998b-60a2c0dc4cee/83bb9cd3-e66c-42fc-8ebd-53e27e95abe3/d3e6b829-08f5-499b-8b35-220ffa9a4993"
 					(reference "#PWR0479")
+					(unit 1)
+				)
+				(path "/090a8e41-87a8-4fb1-998b-60a2c0dc4cee/a33dc8b1-4620-4cf7-8065-8ae8af0e84cf/d3e6b829-08f5-499b-8b35-220ffa9a4993"
+					(reference "#PWR0490")
 					(unit 1)
 				)
@@
 		(on_board yes)
 		(dnp no)
-		(property "Reference" "Q401"
+		(property "Reference" "Q405"
 			(at 151.13 97.7899 0)
 			(effects
@@
 		(instances
 			(project "gpio-module"
-				(path "/090a8e41-87a8-4fb1-998b-60a2c0dc4cee/4ad8e31a-cde3-429e-898f-5d817c85a694/0230d939-768e-429e-8928-f79ac4fd3229"
-					(reference "Q403")
-					(unit 1)
-				)
-				(path "/090a8e41-87a8-4fb1-998b-60a2c0dc4cee/4ad8e31a-cde3-429e-898f-5d817c85a694/05560d46-8ccc-48df-b10d-1c3a365a35b2"
-					(reference "Q402")
-					(unit 1)
-				)
-				(path "/090a8e41-87a8-4fb1-998b-60a2c0dc4cee/4ad8e31a-cde3-429e-898f-5d817c85a694/3200d16b-13e4-4f35-a189-f6ee81970efa"
-					(reference "Q401")
-					(unit 1)
-				)
 				(path "/090a8e41-87a8-4fb1-998b-60a2c0dc4cee/5f7db16d-834d-414e-a24b-79c654644ccf/d3e6b829-08f5-499b-8b35-220ffa9a4993"
 					(reference "Q405")
@@
 					(unit 1)
 				)
+				(path "/090a8e41-87a8-4fb1-998b-60a2c0dc4cee/a33dc8b1-4620-4cf7-8065-8ae8af0e84cf/d3e6b829-08f5-499b-8b35-220ffa9a4993"
+					(reference "Q408")
+					(unit 1)
+				)
