File: mosfet-power-stage.kicad_sch (KiCad schematic)
At the start: 3 parts, among them Q405 AO3400A

Commit message: [#1] Finish PCB
Parts:
- renumbered R427 to R423, R428 to R426
Changed lines of the file:
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@@
 		(on_board yes)
 		(dnp no)
-		(property "Reference" "R427"
+		(property "Reference" "R423"
 			(at 129.54 104.14 0)
 			(effects
@@
 		(instances
 			(project "base-module"
-				(path "/090a8e41-87a8-4fb1-998b-60a2c0dc4cee/1e4742a2-145a-46a6-8222-17374fa3a593/d3e6b829-08f5-499b-8b35-220ffa9a4993"
+				(path "/090a8e41-87a8-4fb1-998b-60a2c0dc4cee/2eacc112-c748-4514-8f19-54a63b484540/d3e6b829-08f5-499b-8b35-220ffa9a4993"
+					(reference "R425")
+					(unit 1)
+				)
+				(path "/090a8e41-87a8-4fb1-998b-60a2c0dc4cee/3ce14170-f6f1-4e98-bfea-8e2751441f01/d3e6b829-08f5-499b-8b35-220ffa9a4993"
 					(reference "R436")
 					(unit 1)
 				)
-				(path "/090a8e41-87a8-4fb1-998b-60a2c0dc4cee/21e14c9e-8cb5-4c0d-8827-cab6b62735cd/d3e6b829-08f5-499b-8b35-220ffa9a4993"
+				(path "/090a8e41-87a8-4fb1-998b-60a2c0dc4cee/482f7d0c-144a-4b8c-8f49-834e199b564c/d3e6b829-08f5-499b-8b35-220ffa9a4993"
+					(reference "R423")
+					(unit 1)
+				)
+				(path "/090a8e41-87a8-4fb1-998b-60a2c0dc4cee/8f334819-7829-459d-a376-c28f1c3582e9/d3e6b829-08f5-499b-8b35-220ffa9a4993"
 					(reference "R429")
-					(unit 1)
-				)
-				(path "/090a8e41-87a8-4fb1-998b-60a2c0dc4cee/b0ae0dc1-1dc3-4071-a986-cf1be8ac718c/d3e6b829-08f5-499b-8b35-220ffa9a4993"
-					(reference "R427")
-					(unit 1)
-				)
-				(path "/090a8e41-87a8-4fb1-998b-60a2c0dc4cee/b5a8ed9d-2492-499d-884c-f314ed804d88/d3e6b829-08f5-499b-8b35-220ffa9a4993"
-					(reference "R431")
 					(unit 1)
 				)
@@
 		(on_board yes)
 		(dnp no)
-		(property "Reference" "R428"
+		(property "Reference" "R426"
 			(at 134.62 96.774 90)
 			(effects
@@
 		(instances
 			(project "base-module"
-				(path "/090a8e41-87a8-4fb1-998b-60a2c0dc4cee/1e4742a2-145a-46a6-8222-17374fa3a593/d3e6b829-08f5-499b-8b35-220ffa9a4993"
+				(path "/090a8e41-87a8-4fb1-998b-60a2c0dc4cee/2eacc112-c748-4514-8f19-54a63b484540/d3e6b829-08f5-499b-8b35-220ffa9a4993"
+					(reference "R427")
+					(unit 1)
+				)
+				(path "/090a8e41-87a8-4fb1-998b-60a2c0dc4cee/3ce14170-f6f1-4e98-bfea-8e2751441f01/d3e6b829-08f5-499b-8b35-220ffa9a4993"
 					(reference "R437")
 					(unit 1)
 				)
-				(path "/090a8e41-87a8-4fb1-998b-60a2c0dc4cee/21e14c9e-8cb5-4c0d-8827-cab6b62735cd/d3e6b829-08f5-499b-8b35-220ffa9a4993"
+				(path "/090a8e41-87a8-4fb1-998b-60a2c0dc4cee/482f7d0c-144a-4b8c-8f49-834e199b564c/d3e6b829-08f5-499b-8b35-220ffa9a4993"
+					(reference "R426")
+					(unit 1)
+				)
+				(path "/090a8e41-87a8-4fb1-998b-60a2c0dc4cee/8f334819-7829-459d-a376-c28f1c3582e9/d3e6b829-08f5-499b-8b35-220ffa9a4993"
 					(reference "R430")
-					(unit 1)
-				)
-				(path "/090a8e41-87a8-4fb1-998b-60a2c0dc4cee/b0ae0dc1-1dc3-4071-a986-cf1be8ac718c/d3e6b829-08f5-499b-8b35-220ffa9a4993"
-					(reference "R428")
-					(unit 1)
-				)
-				(path "/090a8e41-87a8-4fb1-998b-60a2c0dc4cee/b5a8ed9d-2492-499d-884c-f314ed804d88/d3e6b829-08f5-499b-8b35-220ffa9a4993"
-					(reference "R432")
 					(unit 1)
 				)
@@
 		(on_board yes)
 		(dnp no)
-		(property "Reference" "#PWR0480"
+		(property "Reference" "#PWR0481"
 			(at 148.59 116.84 0)
 			(effects
@@
 		(instances
 			(project "base-module"
-				(path "/090a8e41-87a8-4fb1-998b-60a2c0dc4cee/1e4742a2-145a-46a6-8222-17374fa3a593/d3e6b829-08f5-499b-8b35-220ffa9a4993"
-					(reference "#PWR0491")
-					(unit 1)
-				)
-				(path "/090a8e41-87a8-4fb1-998b-60a2c0dc4cee/21e14c9e-8cb5-4c0d-8827-cab6b62735cd/d3e6b829-08f5-499b-8b35-220ffa9a4993"
+				(path "/090a8e41-87a8-4fb1-998b-60a2c0dc4cee/2eacc112-c748-4514-8f19-54a63b484540/d3e6b829-08f5-499b-8b35-220ffa9a4993"
+					(reference "#PWR0483")
+					(unit 1)
+				)
+				(path "/090a8e41-87a8-4fb1-998b-60a2c0dc4cee/3ce14170-f6f1-4e98-bfea-8e2751441f01/d3e6b829-08f5-499b-8b35-220ffa9a4993"
+					(reference "#PWR0487")
+					(unit 1)
+				)
+				(path "/090a8e41-87a8-4fb1-998b-60a2c0dc4cee/482f7d0c-144a-4b8c-8f49-834e199b564c/d3e6b829-08f5-499b-8b35-220ffa9a4993"
 					(reference "#PWR0481")
 					(unit 1)
 				)
-				(path "/090a8e41-87a8-4fb1-998b-60a2c0dc4cee/b0ae0dc1-1dc3-4071-a986-cf1be8ac718c/d3e6b829-08f5-499b-8b35-220ffa9a4993"
-					(reference "#PWR0480")
-					(unit 1)
-				)
-				(path "/090a8e41-87a8-4fb1-998b-60a2c0dc4cee/b5a8ed9d-2492-499d-884c-f314ed804d88/d3e6b829-08f5-499b-8b35-220ffa9a4993"
-					(reference "#PWR0487")
+				(path "/090a8e41-87a8-4fb1-998b-60a2c0dc4cee/8f334819-7829-459d-a376-c28f1c3582e9/d3e6b829-08f5-499b-8b35-220ffa9a4993"
+					(reference "#PWR0485")
 					(unit 1)
 				)
@@
 		(on_board yes)
 		(dnp no)
-		(property "Reference" "#PWR0477"
+		(property "Reference" "#PWR0480"
 			(at 128.27 116.84 0)
 			(effects
@@
 		(instances
 			(project "base-module"
-				(path "/090a8e41-87a8-4fb1-998b-60a2c0dc4cee/1e4742a2-145a-46a6-8222-17374fa3a593/d3e6b829-08f5-499b-8b35-220ffa9a4993"
-					(reference "#PWR0490")
-					(unit 1)
-				)
-				(path "/090a8e41-87a8-4fb1-998b-60a2c0dc4cee/21e14c9e-8cb5-4c0d-8827-cab6b62735cd/d3e6b829-08f5-499b-8b35-220ffa9a4993"
-					(reference "#PWR0479")
-					(unit 1)
-				)
-				(path "/090a8e41-87a8-4fb1-998b-60a2c0dc4cee/b0ae0dc1-1dc3-4071-a986-cf1be8ac718c/d3e6b829-08f5-499b-8b35-220ffa9a4993"
-					(reference "#PWR0477")
-					(unit 1)
-				)
-				(path "/090a8e41-87a8-4fb1-998b-60a2c0dc4cee/b5a8ed9d-2492-499d-884c-f314ed804d88/d3e6b829-08f5-499b-8b35-220ffa9a4993"
+				(path "/090a8e41-87a8-4fb1-998b-60a2c0dc4cee/2eacc112-c748-4514-8f19-54a63b484540/d3e6b829-08f5-499b-8b35-220ffa9a4993"
+					(reference "#PWR0482")
+					(unit 1)
+				)
+				(path "/090a8e41-87a8-4fb1-998b-60a2c0dc4cee/3ce14170-f6f1-4e98-bfea-8e2751441f01/d3e6b829-08f5-499b-8b35-220ffa9a4993"
 					(reference "#PWR0486")
+					(unit 1)
+				)
+				(path "/090a8e41-87a8-4fb1-998b-60a2c0dc4cee/482f7d0c-144a-4b8c-8f49-834e199b564c/d3e6b829-08f5-499b-8b35-220ffa9a4993"
+					(reference "#PWR0480")
+					(unit 1)
+				)
+				(path "/090a8e41-87a8-4fb1-998b-60a2c0dc4cee/8f334819-7829-459d-a376-c28f1c3582e9/d3e6b829-08f5-499b-8b35-220ffa9a4993"
+					(reference "#PWR0484")
 					(unit 1)
 				)
@@
 		(instances
 			(project "base-module"
-				(path "/090a8e41-87a8-4fb1-998b-60a2c0dc4cee/1e4742a2-145a-46a6-8222-17374fa3a593/d3e6b829-08f5-499b-8b35-220ffa9a4993"
+				(path "/090a8e41-87a8-4fb1-998b-60a2c0dc4cee/2eacc112-c748-4514-8f19-54a63b484540/d3e6b829-08f5-499b-8b35-220ffa9a4993"
+					(reference "Q406")
+					(unit 1)
+				)
+				(path "/090a8e41-87a8-4fb1-998b-60a2c0dc4cee/3ce14170-f6f1-4e98-bfea-8e2751441f01/d3e6b829-08f5-499b-8b35-220ffa9a4993"
 					(reference "Q408")
 					(unit 1)
 				)
-				(path "/090a8e41-87a8-4fb1-998b-60a2c0dc4cee/21e14c9e-8cb5-4c0d-8827-cab6b62735cd/d3e6b829-08f5-499b-8b35-220ffa9a4993"
-					(reference "Q406")
-					(unit 1)
-				)
-				(path "/090a8e41-87a8-4fb1-998b-60a2c0dc4cee/b0ae0dc1-1dc3-4071-a986-cf1be8ac718c/d3e6b829-08f5-499b-8b35-220ffa9a4993"
+				(path "/090a8e41-87a8-4fb1-998b-60a2c0dc4cee/482f7d0c-144a-4b8c-8f49-834e199b564c/d3e6b829-08f5-499b-8b35-220ffa9a4993"
 					(reference "Q405")
 					(unit 1)
 				)
-				(path "/090a8e41-87a8-4fb1-998b-60a2c0dc4cee/b5a8ed9d-2492-499d-884c-f314ed804d88/d3e6b829-08f5-499b-8b35-220ffa9a4993"
+				(path "/090a8e41-87a8-4fb1-998b-60a2c0dc4cee/8f334819-7829-459d-a376-c28f1c3582e9/d3e6b829-08f5-499b-8b35-220ffa9a4993"
 					(reference "Q407")
 					(unit 1)
