File: USB.kicad_sch (KiCad schematic)
At the start: 12 parts, among them J800 USB_C_Receptacle_USB2.0_16P, U401 TPD2E2U06DCK, U801 FSUSB42UMX

Commit message: [#1] Fill out schematic title block, connect GPIOs on the schematic
Other:
- title: ModuCard BM STM32H562VGT6 -> ModuCard GPIO module
Changed lines of the file:
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@@
 	(paper "A4")
 	(title_block
-		(title "ModuCard BM STM32H562VGT6")
-		(date "2025-04-18")
-		(rev "1.1.1")
+		(title "ModuCard GPIO module")
+		(date "2025-06-19")
+		(rev "1.0.0")
 		(company "KoNaR")
 		(comment 1 "Base project authors: Dominik Pluta, Artem Horiunov")
-		(comment 2 "Project author: <author>")
+		(comment 2 "Project author: Dominik Pluta")
 	)
 	(junction
