File: base-module.kicad_pcb (KiCad board)
At the start: 4 copper layers, 100 x 100 mm, 166 parts, among them J200 09031967921, J800 USB_C_Receptacle_USB2.0_16P, Q700 MMST3904, U100 W25Q128, U300 TPS563200, U301 TPS563200, U302 CH334P, U401 TPD2E2U06DCK, U402 TPD2E2U06DCK, U403 STM32H562VGTx, U500 TJA1044GTK_3Z, U600 TJA1044GTK_3Z, U700 STM32F103CBTx, U801 FSUSB42UMX, X300 Q13FC1350000400, Y400 ASE-xxxMHz, Y700 Crystal_GND24, Y900 Crystal_GND24

Commit message: [#8] Fix missing component values, fix soldermask expansion of U800 and remove its designator from silkscreen, minor schematic fixes
Parts:
- F300: value Fuse -> 1.5A
- L300, L301: value L -> 3.3uH
- R300: value R_Small -> 54k9
- R306: value R_Small -> 33k2
- R712: value 1.2kΩ -> 1.5kΩ
- Y700: value Crystal_GND24 -> 8 MHz
- Y900: value Crystal_GND24 -> 12Mhz
Changed lines of the file:
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@@
 			)
 		)
-		(property "Value" "L"
+		(property "Value" "3.3uH"
 			(at 0 3.1 90)
 			(layer "F.Fab")
@@
 			)
 		)
-		(property "Description" "Inductor"
+		(property "Description" "DMBJ CXP0420-3R3M-AG(3.3UH)"
 			(at 0 0 90)
 			(layer "F.Fab")
@@
 			)
 		)
-		(property "Value" "R_Small"
+		(property "Value" "33k2"
 			(at 0 0.2 90)
 			(layer "F.Fab")
@@
 			(at -0.041 -1.8104 0)
 			(layer "F.SilkS")
+			(hide yes)
 			(effects
 				(font
@@
 			(pinfunction "D+")
 			(pintype "bidirectional")
-			(solder_mask_margin 0.102)
+			(solder_mask_margin 0.0254)
 		)
 		(pad "2" smd rect
@@
 			(pinfunction "D-")
 			(pintype "bidirectional")
-			(solder_mask_margin 0.102)
+			(solder_mask_margin 0.0254)
 		)
 		(pad "3" smd rect
@@
 			(pinfunction "GND")
 			(pintype "power_in")
-			(solder_mask_margin 0.102)
+			(solder_mask_margin 0.0254)
 		)
 		(pad "4" smd rect
@@
 			(pinfunction "HSD1-")
 			(pintype "input")
-			(solder_mask_margin 0.102)
+			(solder_mask_margin 0.0254)
 		)
 		(pad "5" smd rect
@@
 			(pinfunction "HSD1+")
 			(pintype "input")
-			(solder_mask_margin 0.102)
+			(solder_mask_margin 0.0254)
 		)
 		(pad "6" smd rect
@@
 			(pinfunction "HSD2-")
 			(pintype "input")
-			(solder_mask_margin 0.102)
+			(solder_mask_margin 0.0254)
 		)
 		(pad "7" smd rect
@@
 			(pinfunction "HSD2+")
 			(pintype "input")
-			(solder_mask_margin 0.102)
+			(solder_mask_margin 0.0254)
 		)
 		(pad "8" smd rect
@@
 			(pinfunction "~{OE}")
 			(pintype "input")
-			(solder_mask_margin 0.102)
+			(solder_mask_margin 0.0254)
 		)
 		(pad "9" smd rect
@@
 			(pinfunction "VCC")
 			(pintype "power_in")
-			(solder_mask_margin 0.102)
+			(solder_mask_margin 0.0254)
 		)
 		(pad "10" smd rect
@@
 			(pinfunction "SEL")
 			(pintype "input")
-			(solder_mask_margin 0.102)
+			(solder_mask_margin 0.0254)
 		)
 		(embedded_fonts no)
@@
 			)
 		)
-		(property "Value" "Crystal_GND24"
+		(property "Value" "8 MHz"
 			(at 4.920377 -3.467295 0)
 			(layer "F.Fab")
@@
 			)
 		)
-		(property "Description" "Four pin crystal, GND on pins 2 and 4"
+		(property "Description" "8MHz 20pF ±10ppm SMD3225 Crystals ROHS"
 			(at 0 0 0)
 			(layer "F.Fab")
@@
 			)
 		)
-		(property "Value" "R_Small"
+		(property "Value" "54k9"
 			(at 0 0.2 0)
 			(layer "F.Fab")
@@
 			)
 		)
-		(property "Value" "Fuse"
+		(property "Value" "1.5A"
 			(at 0 1.43 0)
 			(layer "F.Fab")
@@
 			)
 		)
-		(property "Datasheet" ""
+		(property "Datasheet" "https://wmsc.lcsc.com/wmsc/upload/file/pdf/v2/lcsc/2202211730_TLC-Electronic-F06F1-5_C2924957.pdf"
 			(at 0 0 0)
 			(unlocked yes)
@@
 			)
 		)
-		(property "Description" "Fuse"
+		(property "Description" "0603 Disposable fuses ROHS"
 			(at 0 0 0)
 			(unlocked yes)
@@
 			)
 		)
-		(property ki_fp_filters "*Fuse*")
+		(property "LCSC" "C2924957"
+			(at 0 0 0)
+			(unlocked yes)
+			(layer "F.Fab")
+			(hide yes)
+			(effects
+				(font
+					(size 1 1)
+					(thickness 0.15)
+				)
+			)
+		)
+		(property "Stock" "450"
+			(at 0 0 0)
+			(unlocked yes)
+			(layer "F.Fab")
+			(hide yes)
+			(effects
+				(font
+					(size 1 1)
+					(thickness 0.15)
+				)
+			)
+		)
+		(property "Price" "0.048USD"
+			(at 0 0 0)
+			(unlocked yes)
+			(layer "F.Fab")
+			(hide yes)
+			(effects
+				(font
+					(size 1 1)
+					(thickness 0.15)
+				)
+			)
+		)
+		(property "Process" "SMT"
+			(at 0 0 0)
+			(unlocked yes)
+			(layer "F.Fab")
+			(hide yes)
+			(effects
+				(font
+					(size 1 1)
+					(thickness 0.15)
+				)
+			)
+		)
+		(property "Minimum Qty" "5"
+			(at 0 0 0)
+			(unlocked yes)
+			(layer "F.Fab")
+			(hide yes)
+			(effects
+				(font
+					(size 1 1)
+					(thickness 0.15)
+				)
+			)
+		)
+		(property "Attrition Qty" "4"
+			(at 0 0 0)
+			(unlocked yes)
+			(layer "F.Fab")
+			(hide yes)
+			(effects
+				(font
+					(size 1 1)
+					(thickness 0.15)
+				)
+			)
+		)
+		(property "Class" "Preferred Component"
+			(at 0 0 0)
+			(unlocked yes)
+			(layer "F.Fab")
+			(hide yes)
+			(effects
+				(font
+					(size 1 1)
+					(thickness 0.15)
+				)
+			)
+		)
+		(property "Category" "TVS/Fuse/Board Level Protection,Fuses"
+			(at 0 0 0)
+			(unlocked yes)
+			(layer "F.Fab")
+			(hide yes)
+			(effects
+				(font
+					(size 1 1)
+					(thickness 0.15)
+				)
+			)
+		)
+		(property "Manufacturer" "TLC Electronic"
+			(at 0 0 0)
+			(unlocked yes)
+			(layer "F.Fab")
+			(hide yes)
+			(effects
+				(font
+					(size 1 1)
+					(thickness 0.15)
+				)
+			)
+		)
+		(property "Part" "F06F1.5"
+			(at 0 0 0)
+			(unlocked yes)
+			(layer "F.Fab")
+			(hide yes)
+			(effects
+				(font
+					(size 1 1)
+					(thickness 0.15)
+				)
+			)
+		)
+		(property ki_fp_filters "F_*")
 		(sheetname "/Power/")
 		(sheetfile "power.kicad_sch")
@@
 			)
 		)
-		(property "Value" "1.2kΩ"
+		(property "Value" "1.5kΩ"
 			(at 0 0.199999 135)
 			(layer "F.Fab")
@@
 			)
 		)
-		(property "Datasheet" "https://www.lcsc.com/datasheet/lcsc_datasheet_2206010045_UNI-ROYAL-Uniroyal-Elec-0402WGF1201TCE_C25862.pdf"
+		(property "Datasheet" "https://www.lcsc.com/datasheet/lcsc_datasheet_2206010045_UNI-ROYAL-Uniroyal-Elec-0402WGF1501TCE_C25867.pdf"
 			(at 0 0 135)
 			(unlocked yes)
@@
 			)
 		)
-		(property "Description" "62.5mW Thick Film Resistors 50V ±100ppm/°C ±1% 1.2kΩ 0402 Chip Resistor - Surface Mount ROHS"
+		(property "Description" "62.5mW Thick Film Resistors 50V ±100ppm/°C ±1% 1.5kΩ 0402 Chip Resistor - Surface Mount ROHS"
 			(at 0 0 135)
 			(unlocked yes)
@@
 			)
 		)
-		(property "LCSC" "C25862"
+		(property "LCSC" "C25867"
 			(at 0 0 135)
 			(unlocked yes)
@@
 			)
 		)
-		(property "Stock" "191144"
+		(property "Stock" "853285"
 			(at 0 0 135)
 			(unlocked yes)
@@
 			)
 		)
-		(property "Class" "Preferred Component"
+		(property "Class" "Basic Component"
 			(at 0 0 135)
 			(unlocked yes)
@@
 			)
 		)
-		(property "Part" "0402WGF1201TCE"
+		(property "Part" "0402WGF1501TCE"
 			(at 0 0 135)
 			(unlocked yes)
@@
 			)
 		)
-		(property "Resistance" "1.2kΩ"
+		(property "Resistance" "1.5kΩ"
 			(at 0 0 135)
 			(unlocked yes)
@@
 			)
 		)
-		(property "Value" "Crystal_GND24"
+		(property "Value" "12Mhz"
 			(at 0 2.45 0)
 			(layer "F.Fab")
@@
 			)
 		)
-		(property "Description" "Four pin crystal, GND on pins 2 and 4"
+		(property "Description" ""
 			(at 0 0 180)
 			(unlocked yes)
@@
 			)
 		)
-		(property "Value" "L"
+		(property "Value" "3.3uH"
 			(at 1.692256 6.083788 0)
 			(layer "F.Fab")
@@
 			)
 		)
-		(property "Description" "Inductor"
+		(property "Description" "DMBJ CXP0420-3R3M-AG(3.3UH)"
 			(at 0 0 0)
 			(layer "F.Fab")
@@
 		(layer "F.Cu")
 		(net 1)
-	)
-	(segment
-		(start 120.888001 109.375)
-		(end 120.888 109.375001)
-		(width 0.15)
-		(layer "F.Cu")
-		(net 1)

Commit message: [#8] Fix LEDs resistors values
Parts:
- removed R400: 1.2kΩ, PCM_JLCPCB:R_0402
- removed R408: 220Ω, PCM_JLCPCB:R_0402
- removed R409: 100Ω, PCM_JLCPCB:R_0402
- added R414: 220Ω, PCM_JLCPCB:R_0402, F.Cu at (114.5, 61.2)
- added R415: 220Ω, PCM_JLCPCB:R_0402, F.Cu at (115.3, 61.2)
- added R416: 220Ω, PCM_JLCPCB:R_0402, F.Cu at (113.5, 61.2)

Commit message: [#8] Bump project to rev.1.1.1
Other:
- board text added: "PROJECT Rev. 1.0.0 TEMPLATE Rev. 1.1.1"
- board text removed: "PROJECT Rev. 1.0.0 TEMPLATE Rev. 1.1.0"
Changed lines of the file:
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@@
 		(title "ModuCard base module")
 		(date "2025-02-25")
-		(rev "1.1.0")
+		(rev "1.1.1")
 		(company "KoNaR")
 		(comment 1 "Base project author: Dominik Pluta Artem Horiunov")
@@
 		)
 	)
-	(gr_text "PROJECT  Rev. 1.0.0\nTEMPLATE Rev. 1.1.0\n"
+	(gr_text "PROJECT  Rev. 1.0.0\nTEMPLATE Rev. 1.1.1\n"
 		(at 118.97 74.085001 0)
 		(layer "F.SilkS")

Commit message: [#1] Finish PCB
Parts:
- added F301: Fuse, PCM_JLCPCB:R_0603, F.Cu at (45.2, 62.2)
- added J10: Molex_Micro-Fit_3.0 2x2, Connector_Molex:Molex_Micro-Fit_3.0_43045-0400_2x02_P3.00mm_Horizontal, F.Cu at (66.1, 60.5)
- added J11: Molex_Micro-Fit_3.0 2x2, Connector_Molex:Molex_Micro-Fit_3.0_43045-0400_2x02_P3.00mm_Horizontal, F.Cu at (54.9, 60.5)
- added J8: Molex_Micro-Fit_3.0 2x2, Connector_Molex:Molex_Micro-Fit_3.0_43045-0400_2x02_P3.00mm_Horizontal, F.Cu at (88.7, 60.5)
- added J9: Molex_Micro-Fit_3.0 2x2, Connector_Molex:Molex_Micro-Fit_3.0_43045-0400_2x02_P3.00mm_Horizontal, F.Cu at (77.4, 60.5)
- added Q405: AO3400A, PCM_JLCPCB:Q_SOT-23, F.Cu at (80.4, 69.5)
- added Q406: AO3400A, PCM_JLCPCB:Q_SOT-23, F.Cu at (69.1, 69.5)
- added Q407: AO3400A, PCM_JLCPCB:Q_SOT-23, F.Cu at (57.9, 69.5)
- added Q408: AO3400A, PCM_JLCPCB:Q_SOT-23, F.Cu at (91.7, 69.5)
- added R400: 10kΩ, PCM_JLCPCB:R_0402, F.Cu at (77.4, 68.5)
- added R417: 10kΩ, PCM_JLCPCB:R_0402, F.Cu at (66.1, 68.5)
- added R418: 10kΩ, PCM_JLCPCB:R_0402, F.Cu at (54.9, 68.5)
- added R419: 10kΩ, PCM_JLCPCB:R_0402, F.Cu at (88.7, 68.5)
- added R420: 22kΩ, PCM_JLCPCB:R_0402, F.Cu at (77.4, 70.5)
- added R421: 22kΩ, PCM_JLCPCB:R_0402, F.Cu at (66.1, 70.5)
- added R422: 22kΩ, PCM_JLCPCB:R_0402, F.Cu at (54.9, 70.4)
- added R423: 10kΩ, PCM_JLCPCB:R_0402, F.Cu at (80.4, 71.9)
- added R424: 22kΩ, PCM_JLCPCB:R_0402, F.Cu at (88.7, 70.4)
- added R425: 10kΩ, PCM_JLCPCB:R_0402, F.Cu at (69.1, 71.9)
- added R426: 100Ω, PCM_JLCPCB:R_0402, F.Cu at (80.4, 72.7)
- added R427: 100Ω, PCM_JLCPCB:R_0402, F.Cu at (69.1, 72.7)
- added R429: 10kΩ, PCM_JLCPCB:R_0402, F.Cu at (57.9, 71.9)
- added R430: 100Ω, PCM_JLCPCB:R_0402, F.Cu at (57.9, 72.7)
- added R436: 10kΩ, PCM_JLCPCB:R_0402, F.Cu at (91.7, 71.9)
- added R437: 100Ω, PCM_JLCPCB:R_0402, F.Cu at (91.7, 72.7)
- added TP303: TestPoint, TestPoint:TestPoint_Pad_D1.0mm, F.Cu at (50.4, 63.3)
- added kibuzzard-682A47D8: G***, kibuzzard-682A47D8, F.Cu at (50.4, 67.2)
Connections:
- U403 pad 16: unconnected-(U403-PC1-Pad16) -> /GPIO connector 3/input
- U403 pad 17: unconnected-(U403-PC2-Pad17) -> /GPIO connector 3/output
- U403 pad 18: unconnected-(U403-PC3-Pad18) -> /GPIO connector 0/output
- U403 pad 23: unconnected-(U403-PA0-Pad23) -> /GPIO connector 0/input
- U403 pad 24: unconnected-(U403-PA1-Pad24) -> /GPIO connector 1/output
- U403 pad 25: unconnected-(U403-PA2-Pad25) -> /GPIO connector 1/input
- U403 pad 26: unconnected-(U403-PA3-Pad26) -> /GPIO connector 2/output
- U403 pad 29: unconnected-(U403-PA4-Pad29) -> /GPIO connector 2/input
- U403 pad 30: unconnected-(U403-PA5-Pad30) -> /Backplane/GPIOR15
- U403 pad 31: unconnected-(U403-PA6-Pad31) -> /Backplane/GPIOR14
- U403 pad 32: unconnected-(U403-PA7-Pad32) -> /Backplane/GPIOR13
- U403 pad 33: unconnected-(U403-PC4-Pad33) -> /Backplane/GPIOR12
- U403 pad 34: unconnected-(U403-PC5-Pad34) -> /Backplane/GPIOR11
- U403 pad 35: unconnected-(U403-PB0-Pad35) -> /Backplane/GPIOR10
- U403 pad 36: unconnected-(U403-PB1-Pad36) -> /Backplane/GPIOR9
- U403 pad 38: unconnected-(U403-PE7-Pad38) -> /Backplane/GPIOR8
- U403 pad 39: unconnected-(U403-PE8-Pad39) -> /Backplane/GPIOR7
- U403 pad 40: unconnected-(U403-PE9-Pad40) -> /Backplane/GPIOR6
- U403 pad 41: unconnected-(U403-PE10-Pad41) -> /Backplane/GPIOR5
- U403 pad 42: unconnected-(U403-PE11-Pad42) -> /Backplane/GPIOR4
- U403 pad 43: unconnected-(U403-PE12-Pad43) -> /Backplane/GPIOR3
- U403 pad 44: unconnected-(U403-PE13-Pad44) -> /Backplane/GPIOR2
- U403 pad 45: unconnected-(U403-PE14-Pad45) -> /Backplane/GPIOR1
- U403 pad 46: unconnected-(U403-PE15-Pad46) -> /Backplane/GPIOR0
- U403 pad 53: unconnected-(U403-PB14-Pad53) -> /Backplane/GPIOL15
- U403 pad 54: unconnected-(U403-PB15-Pad54) -> /Backplane/GPIOL14
- U403 pad 55: unconnected-(U403-PD8-Pad55) -> /Backplane/GPIOL13
- U403 pad 56: unconnected-(U403-PD9-Pad56) -> /Backplane/GPIOL12
- U403 pad 57: unconnected-(U403-PD10-Pad57) -> /Backplane/GPIOL11
- U403 pad 61: unconnected-(U403-PD14-Pad61) -> /Backplane/GPIOL10
- U403 pad 62: unconnected-(U403-PD15-Pad62) -> /Backplane/GPIOL9
- U403 pad 63: unconnected-(U403-PC6-Pad63) -> /Backplane/GPIOL8
- U403 pad 64: unconnected-(U403-PC7-Pad64) -> /Backplane/GPIOL7
- U403 pad 65: unconnected-(U403-PC8-Pad65) -> /Backplane/GPIOL6
- U403 pad 66: unconnected-(U403-PC9-Pad66) -> /Backplane/GPIOL5
- U403 pad 67: unconnected-(U403-PA8-Pad67) -> /Backplane/GPIOL4
- U403 pad 68: unconnected-(U403-PA9-Pad68) -> /Backplane/GPIOL3
- U403 pad 69: unconnected-(U403-PA10-Pad69) -> /Backplane/GPIOL2
- U403 pad 78: unconnected-(U403-PC10-Pad78) -> /Backplane/GPIOL1
- U403 pad 79: unconnected-(U403-PC11-Pad79) -> /Backplane/GPIOL0
Routing:
- net +5V: track 38.2 -> 167.0 mm, vias 10 -> 14
- net /GPIO connector 2/input: track 0.00 -> 84.9 mm, vias 0 -> 2
- net /GPIO connector 2/output: track 0.00 -> 76.4 mm, vias 0 -> 2
- net /Backplane/GPIOL15: track 0.00 -> 74.2 mm, vias 0 -> 1
- net /Backplane/GPIOL14: track 0.00 -> 70.4 mm, vias 0 -> 1
- net /GPIO connector 1/input: track 0.00 -> 69.5 mm, vias 0 -> 2
- net /Backplane/GPIOL13: track 0.00 -> 68.6 mm, vias 0 -> 1
- net /Backplane/GPIOR15: track 0.00 -> 66.3 mm, vias 0 -> 1
- net /GPIO connector 1/output: track 0.00 -> 65.3 mm, vias 0 -> 2
- net /Backplane/GPIOL12: track 0.00 -> 65.2 mm, vias 0 -> 1
- net /Backplane/GPIOL10: track 0.00 -> 64.4 mm, vias 0 -> 1
- net /Backplane/GPIOR14: track 0.00 -> 63.5 mm, vias 0 -> 1
- net /GPIO connector 0/input: track 0.00 -> 63.5 mm, vias 0 -> 2
- net /Backplane/GPIOL11: track 0.00 -> 63.5 mm, vias 0 -> 1
- net /Backplane/GPIOR13: track 0.00 -> 61.5 mm, vias 0 -> 1
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- added copper zone on F.Cu, net +12V_GPIO
Other:
- board text added: "12V"
- board text added: "12V FUSE"
- board text added: "5V"
- board text added: "CH0"
- board text added: "CH1"
- board text added: "CH2"
- board text added: "CH3"
- board text added: "F PANEL"
- board text added: "GPIO"
- board text added: "MAIN MODULE"
- board text removed: "* HIGH PERFORMANCE MCU * ADDITIONAL (Q)SPI FLASH * BUILT IN USB DEBUGGER * HIGH SPEED CAN TANSCEIVERS * HIGH POWER 24W VRM"
- board text removed: "1. Add $Project Author$ field 2. Add board revision 3. Remove this silkscreen 4. Layout board 6. Pass DRC 5. Add boardhouse info in designted spot on bottom side"
- board text removed: "BY NOMAD ELECTRONICS TEAM"
- board text removed: "FEATURES:"
- board text removed: "Template Project"
- board text removed: "USAGE:"
- board text removed: "USER AREA"
- board text removed: "predefined area"
