File: base-module.kicad_sch (KiCad schematic)
At the start: 0 parts

Commit message: [#1] Fill out schematic title block, connect GPIOs on the schematic
Connections:
- no-connect marks 3 -> 1
Other:
- added sheet GPIO connector 0 (gpio-connector.kicad_sch)
- added sheet GPIO connector 1 (gpio-connector.kicad_sch)
- added sheet GPIO connector 2 (gpio-connector.kicad_sch)
- added sheet GPIO connector 3 (gpio-connector.kicad_sch)
- sheet MCU ports: added GPIOL[0..15], GPIOR[0..15], GPIO_0_IN, GPIO_0_OUT, GPIO_1_IN, GPIO_1_OUT, GPIO_2_IN, GPIO_2_OUT, GPIO_3_IN, GPIO_3_OUT; removed none
- title: ModuCard BM STM32H562VGT6 -> ModuCard GPIO module
